File: PCBs/MainPCB/microstim.kicad_pcb (KiCad board)
At the start: 2 copper layers, 124.5 x 79.5 mm, 103 parts, among them J1 Conn_Coaxial, J10 Conn_Coaxial, J11 Screw_Terminal_01x02, J12 Conn_Coaxial, J2 Conn_02x08_Counter_Clockwise, J3 Screw_Terminal_01x02, J5 Conn_Coaxial, J7 Screw_Terminal_01x02, J9 Screw_Terminal_01x02, SW1 SW_Push, U1 Teensy3.5, U10 AD7321, U11 INA826, U12 AD8276, U13 AD8276, U14 INA826, U15 OPA197, U16 DG509ACWE, U17 OPA197, U18 DG509ACWE, U19 ISO7341C, U2 CC3-0512DF-E, U20 L78L05_SO8, U21 AD5752, U22 AD7321, U23 AD1582, U3 L78L05_SO8, U4 AD5752, U5 ISO7760, U6 AD1582, U7 ISO7341C, U8 CC3-0512DF-E, U9 ISO7760

Commit message: making progress on layout... slowly
Parts:
- removed the C2 at (170.9, 106.2)
- removed the C27 at (149.2, 69.6)
- removed the C28 at (152.6, 80.8)
- removed the C31 at (166.3, 85.1)
- removed the C33 at (169.3, 90.2)
- removed the C36 at (161.7, 80.5)
- removed the C40 at (160.9, 69.6)
- removed the C49 at (224.5, 118.3)
- removed the C9 at (160.0, 116.0)
- removed J10: Conn_Coaxial, microstim:731375003
- removed the R13 at (166.3, 79.7)
- removed R15: 1k, Resistor_SMD:R_0603_1608Metric
- removed R17: 500, Resistor_SMD:R_0603_1608Metric
- removed the U15 at (150.6, 74.8)
- removed the U18 at (163.6, 74.8)
- removed the U3 at (169.8, 109.7)
- removed the U7 at (167.2, 119.4)
- removed the U8 at (194.0, 130.0)
- added C12: 1uF, Capacitor_SMD:C_0603_1608Metric, F.Cu at (159.7, 86.4)
- added C18: 0.1uF, Capacitor_SMD:C_0603_1608Metric, F.Cu at (124.7, 72.7)
- added C19: 0.1uF, Capacitor_SMD:C_0603_1608Metric, F.Cu at (131.2, 72.6)
- added C22: 0.1uF, Capacitor_SMD:C_0603_1608Metric, F.Cu at (159.8, 77.2)
- added C23: 0.1uF, Capacitor_SMD:C_0603_1608Metric, F.Cu at (145.7, 81.9)
- added C24: 0.1uF, Capacitor_SMD:C_0603_1608Metric, F.Cu at (139.3, 80.6)
- added C25: 0.1uF, Capacitor_SMD:C_0603_1608Metric, F.Cu at (149.6, 77.9)
- added C34: 0.1uF, Capacitor_SMD:C_0603_1608Metric, F.Cu at (186.3, 96.7)
- added C51: 1uF, Capacitor_SMD:C_0603_1608Metric, F.Cu at (123.2, 95.0)
- added C52: 1uF, Capacitor_SMD:C_0603_1608Metric, F.Cu at (167.6, 94.6)
- added C8: 1uF, Capacitor_SMD:C_0603_1608Metric, F.Cu at (149.5, 85.6)
- added J7: Conn_Coaxial, microstim:731375003, F.Cu at (161.3, 59.7)
- added R2: 3k, Resistor_SMD:R_0603_1608Metric, F.Cu at (132.5, 83.0)
- added R4: 3k, Resistor_SMD:R_0603_1608Metric, F.Cu at (136.7, 77.2)
- added R6: 1.8k, Resistor_SMD:R_0603_1608Metric, F.Cu at (143.0, 72.4)
- added U10: AD8276, Package_SO:SOIC-8_3.9x4.9mm_P1.27mm, F.Cu at (132.6, 77.3)
- added U13: CC3-0512DF-E, microstim:CC3-0512DF-E, F.Cu at (205.5, 112.5)
- added U4: ISO7341C, Package_SO:SOIC-16W_7.5x10.3mm_P1.27mm, F.Cu at (126.0, 107.9)
- added U5: L78L05_SO8, Package_SO:SOIC-8_3.9x4.9mm_P1.27mm, F.Cu at (154.2, 84.5)
- added U9: OPA197, Package_SO:SOIC-8_3.9x4.9mm_P1.27mm, F.Cu at (126.1, 77.4)
- C1: renamed from C3; moved to F.Cu
- C2: renamed from C5; moved to F.Cu
- C28: renamed from C32; moved to B.Cu
- C29: renamed from C34; moved to B.Cu
- C3: renamed from C1; moved to B.Cu
- C30: renamed from C35; moved to B.Cu
- C4: renamed from C10; moved to B.Cu
- C5: renamed from C26; moved to B.Cu
- C6: renamed from C11; moved to F.Cu
- C7: value 1uF -> 0.1uF
- R1: value 3k -> 1k
- R3: value 100 -> 500
- R5: value 3k -> 100
- R7: value 1.8k -> 1k
- U12: value AD8276 -> DG509ACWE; footprint Package_SO:SOIC-8_3.9x4.9mm_P1.27mm -> Package_SO:SOIC-16_3.9x9.9mm_P1.27mm
- U14: renamed from U9; moved to F.Cu
- U15: renamed from U19; moved to F.Cu
- U3: renamed from U5; moved to F.Cu
- moved C14 82.0 mm to (132.9, 85.7), turned to 270 degrees
- moved SW1 71.0 mm to (109.1, 146.5)
- moved C35 65.2 mm to (169.6, 94.6), turned to 90 degrees
- moved C31 61.9 mm to (166.7, 101.2)
- moved C38 59.8 mm to (172.1, 86.3), turned to 180 degrees
- moved C6 53.6 mm to (122.0, 101.3), turned to 0 degrees
- moved C2 52.6 mm to (122.3, 114.5), turned to 0 degrees
- moved C39 50.9 mm to (177.6, 85.6), turned to 270 degrees
- moved C26 50.1 mm to (177.8, 114.6), turned to 180 degrees
- moved C42 48.4 mm to (184.3, 85.2), turned to 90 degrees
- moved C36 48.1 mm to (184.7, 96.7), turned to 270 degrees
- moved C27 48.1 mm to (166.8, 114.7)
- moved J4 48.0 mm to (74.5, 58.0)
- moved C37 45.1 mm to (203.9, 86.9), turned to 180 degrees
- moved C40 43.1 mm to (175.9, 85.6), turned to 270 degrees
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- renumbered C42 to C10, C4 to C11, C8 to C13, C15 to C14, C12 to C15, C6 to C26, C14 to C27, C37 to C31, C38 to C32, C39 to C33, C44 to C35, C43 to C36, C45 to C37, C46 to C38, C47 to C39, C48 to C40, C50 to C42, C29 to C43, C30 to C44, C18 to C45, C19 to C46, C24 to C47, C22 to C48, C23 to C49, C25 to C50, C13 to C9, J2 to J1, J5 to J2, J1 to J3, J7 to J4, J3 to J5, J9 to J6, J11 to J8, J12 to J9, R18 to R10, R4 to R11, R6 to R12, R8 to R13, R9 to R14, R16 to R8, R2 to R9, U20 to U16, U21 to U17, U22 to U18, U23 to U19, U17 to U20, U13 to U21, U14 to U22, U16 to U23, U4 to U6, U10 to U7, U6 to U8
Connections:
- C20 pad 1: -15V -> -15V_0
- C21 pad 1: GND_0 -> -15V_0
- C21 pad 2: +15V -> GND_0
- C41 pad 1: -15V_1 -> +15V_1
- C43 pad 1: GNDREF -> GND_1
- C43 pad 2: +15V -> +15V_1
- C44 pad 1: -15V -> -15V_1
- C44 pad 2: GNDREF -> GND_1
- C45 pad 1: GNDREF -> GND_1
- C45 pad 2: +15V -> +15V_1
- C46 pad 1: -15V -> -15V_1
- C46 pad 2: GNDREF -> GND_1
- C47 pad 1: GNDREF -> GND_1
- C47 pad 2: -15V -> -15V_1
- C48 pad 1: GNDREF -> GND_1
- C48 pad 2: +15V -> +15V_1
- C49 pad 1: GNDREF -> GND_1
- C49 pad 2: -15V -> -15V_1
- C50 pad 1: GNDREF -> GND_1
- C50 pad 2: +15V -> +15V_1
- J2 pad 1: Net-(J5-Pad1) -> Net-(J2-Pad1)
- J4 pad 1: Net-(J5-Pad1) -> Net-(J2-Pad1)
- J6 pad 2: GNDREF -> GND_0
- J8 pad 2: GNDREF -> GND_1
- J9 pad 2: GNDREF -> GND_1
- R1 pad 1: Net-(R1-Pad1) -> GND_0
- R1 pad 2: DAC_0 -> Net-(R1-Pad2)
- R14 pad 1: GNDREF -> GND_1
- R3 pad 1: Net-(R3-Pad1) -> Net-(R1-Pad2)
- R3 pad 2: IOUT_0 -> VOUT_0
- R5 pad 1: Net-(R3-Pad1) -> Net-(R4-Pad1)
- R5 pad 2: Net-(R5-Pad2) -> IOUT_0
- R7 pad 2: Net-(R7-Pad2) -> GND_0
- R8 pad 1: GNDREF -> GND_1
- U1 pad 13: MOSI_0 -> MOSI
- U1 pad 14: MISO_0 -> MISO
- U1 pad 2: MOSI_1 -> Net-(U1-Pad2)
- U1 pad 24: SCK_1 -> Net-(U1-Pad24)
- U1 pad 3: MISO_1 -> Net-(U1-Pad3)
- U1 pad 40: SCK_0 -> SCK
- U1 pad 50: GND -> Net-(J2-Pad1)
- U11 pad 2: Net-(R7-Pad2) -> Net-(R6-Pad2)
- U11 pad 3: Net-(R7-Pad1) -> Net-(R6-Pad1)
- U11 pad 4: Net-(R3-Pad1) -> Net-(R4-Pad1)
- U11 pad 5: -15V -> -15V_0
- U11 pad 6: GNDREF -> GND_0
- U11 pad 8: +15V -> +15V_0
- U12 pad 1: Net-(R3-Pad1) -> OE0_0i
- U12 pad 2: GND_0 -> +5V_0
- U12 pad 3: Net-(R1-Pad1) -> -15V_0
- U12 pad 4: -15V -> Net-(R7-Pad1)
- U12 pad 5: Net-(R5-Pad2) -> Net-(U12-Pad12)
- U12 pad 6: Net-(R5-Pad2) -> Net-(U12-Pad11)
- U12 pad 7: +15V -> Net-(R7-Pad1)
- U12 pad 8: Net-(U12-Pad8) -> IOUT_0
- U15 pad 3: MOSI_1 -> MOSI
- U15 pad 4: SCK_1 -> SCK
- U15 pad 6: MISO_1 -> MISO
- U20 pad 4: -15V -> -15V_1
- U20 pad 7: +15V -> +15V_1
- U21 pad 2: GNDREF -> GND_1
- U21 pad 4: -15V -> -15V_1
- U21 pad 7: +15V -> +15V_1
- U22 pad 5: -15V -> -15V_1
- U22 pad 6: GNDREF -> GND_1
- U22 pad 8: +15V -> +15V_1
- U23 pad 10: GNDREF -> GND_1
- U23 pad 14: +15V -> +15V_1
- U23 pad 15: GNDREF -> GND_1
- U23 pad 2: +5V -> +5V_1
- U23 pad 3: -15V -> -15V_1
Routing:
- net +5V_0: track 0.00 -> 139.2 mm, vias 0 -> 8
- net +15V: track 117.0 -> 0.00 mm, vias 9 -> 0
- net -15V_0: track 0.00 -> 109.8 mm, vias 0 -> 5
- net -15V: track 90.6 -> 0.00 mm, vias 8 -> 0
- net +15V_0: track 0.00 -> 88.7 mm, vias 0 -> 7
- net Net-(J3-Pad1): track 85.9 -> 0.00 mm
- net Net-(J5-Pad1): track 80.5 -> 0.00 mm
- net Net-(J1-Pad15): track 53.3 -> 0.00 mm
- net Net-(J1-Pad14): track 53.2 -> 0.00 mm
- net GNDREF: track 49.8 -> 0.00 mm, vias 10 -> 0
- net Net-(J1-Pad13): track 47.2 -> 0.00 mm
- net Net-(J1-Pad12): track 47.1 -> 0.00 mm
- net +5V: track 42.2 -> 0.00 mm, vias 3 -> 0
- net Net-(J1-Pad10): track 39.1 -> 0.00 mm
- net Net-(J1-Pad11): track 38.5 -> 0.00 mm
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
Commit message: getting darn close to done with layout.
Parts:
- J1: value Conn_02x08_Counter_Clockwise -> Conn_02x08_Odd_Even
- moved D2 71.3 mm to (127.7, 127.1)
- moved D1 47.0 mm to (120.5, 127.1)
- moved J1 43.9 mm to (168.1, 121.3)
- moved SW1 19.9 mm to (111.5, 126.7)
- moved C48 13.5 mm to (190.7, 81.4), turned to 180 degrees
- moved J2 2.80 mm to (121.3, 59.5)
- moved R13 1.46 mm to (188.0, 71.7)
- moved U1 1.30 mm to (94.8, 99.9)
- moved J3 1.20 mm to (100.4, 59.4)
- moved R11 1.17 mm to (181.6, 76.9)
- moved R8 1.17 mm to (169.3, 81.5)
- moved C44 1.17 mm to (173.6, 81.6)
- moved R10 1.17 mm to (166.6, 76.6)
- moved U21 1.17 mm to (177.6, 76.8)
- moved U22 1.17 mm to (188.0, 76.7)
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Connections:
- J1 pad 1: GND -> +3V3
- J1 pad 10: Net-(J1-Pad10) -> GPIO8
- J1 pad 11: Net-(J1-Pad11) -> GPIO3
- J1 pad 12: Net-(J1-Pad12) -> GPIO9
- J1 pad 13: Net-(J1-Pad13) -> GPIO4
- J1 pad 14: Net-(J1-Pad14) -> GPIO10
- J1 pad 15: Net-(J1-Pad15) -> GPIO5
- J1 pad 16: Net-(J1-Pad16) -> GPIO11
- J1 pad 3: GPIO0 -> GND
- J1 pad 4: GPIO1 -> GND
- J1 pad 5: GPIO2 -> GPIO0
- J1 pad 6: GPIO3 -> GPIO6
- J1 pad 7: GPIO4 -> GPIO1
- J1 pad 8: GPIO5 -> GPIO7
- J1 pad 9: GND -> GPIO2
- U1 pad 10: OE0_0 -> CS1_0
- U1 pad 11: CS1_0 -> CS0_0
- U1 pad 12: CS0_0 -> NLDAC_0
- U1 pad 16: NLDAC_0 -> Net-(U1-Pad16)
- U1 pad 3: Net-(U1-Pad3) -> OE1_1
- U1 pad 32: Net-(J1-Pad15) -> Net-(U1-Pad32)
- U1 pad 33: Net-(J1-Pad14) -> GPIO0
- U1 pad 34: Net-(J1-Pad13) -> GPIO1
- U1 pad 35: Net-(J1-Pad12) -> GPIO2
- U1 pad 36: Net-(U1-Pad36) -> GPIO3
- U1 pad 37: Net-(J1-Pad11) -> GPIO4
- U1 pad 38: Net-(J1-Pad10) -> GPIO5
- U1 pad 4: OE1_1 -> OE0_1
- U1 pad 43: GPIO5 -> GPIO11
- U1 pad 44: GPIO4 -> GPIO10
- U1 pad 45: GPIO3 -> GPIO9
- U1 pad 46: GPIO2 -> GPIO8
- U1 pad 47: GPIO1 -> GPIO7
- U1 pad 48: GPIO0 -> GPIO6
- U1 pad 5: OE0_1 -> CS1_1
- U1 pad 6: CS1_1 -> CS0_1
- U1 pad 7: CS0_1 -> NLDAC_1
- U1 pad 8: NLDAC_1 -> OE1_0
- U1 pad 9: OE1_0 -> OE0_0
Routing:
- net VUSB: track 0.00 -> 178.1 mm
- net +5V_1: track 0.00 -> 133.0 mm, vias 0 -> 8
- net +3V3: track 0.00 -> 122.6 mm, vias 0 -> 7
- net -15V_1: track 0.00 -> 110.5 mm, vias 0 -> 5
- net SCK: track 0.00 -> 98.8 mm
- net GPIO0: track 0.00 -> 96.9 mm
- net GPIO1: track 0.00 -> 93.2 mm
- net OE1_1: track 0.00 -> 89.3 mm
- net GPIO2: track 0.00 -> 88.6 mm
- net MISO: track 0.00 -> 88.2 mm, vias 0 -> 3
- net +15V_1: track 0.00 -> 87.3 mm, vias 0 -> 6
- net OE0_1: track 0.00 -> 86.8 mm
- net CS1_1: track 0.00 -> 84.9 mm
- net GPIO3: track 0.00 -> 84.3 mm
- net GPIO6: track 0.00 -> 84.0 mm
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
Commit message: finished layout, schematic+pcb pdfs, BOM. need to do panels.
Parts:
- removed J4, J5: Screw_Terminal_01x02, microstim:1-2834016-2 _TERM_BLK_2P_SIDE_ENT_2.54MM_PCB
- added R15: 200, Resistor_SMD:R_0603_1608Metric, F.Cu at (117.5, 126.4)
- added R16: 200, Resistor_SMD:R_0603_1608Metric, F.Cu at (127.7, 126.3)
- D1, D2: footprint LED_THT:LED_D5.0mm_Horizontal_O1.27mm_Z3.0mm -> microstim:LED_D5.0mm_Horizontal_O1.27mm_Z3.0mm_pinSwapped
- SW1: footprint Button_Switch_SMD:SW_SPST_EVPBF -> microstim:EVQ-PF303K
- moved H4 127.8 mm to (200.0, 125.0)
- moved H1 106.8 mm to (170.0, 60.0)
- moved H2 60.9 mm to (128.0, 60.0)
- moved H3 33.7 mm to (110.0, 85.0)
- moved J2 20.6 mm to (100.7, 59.5)
- moved J3 20.4 mm to (120.8, 59.5)
- moved D2 3.35 mm to (131.0, 126.5)
- moved SW1 2.47 mm to (109.4, 125.4)
- moved D1 0.60 mm to (120.5, 126.5)
Connections:
- D1 pad 1: Net-(D1-Pad1) -> GND
- D2 pad 1: Net-(D2-Pad1) -> GND
- J1 pad 1: +3V3 -> GND
- J1 pad 3: GND -> +3V3
- U1 pad 41: Net-(U1-Pad41) -> GPIO11
- U1 pad 42: Net-(U1-Pad42) -> GPIO10
- U1 pad 43: GPIO11 -> GPIO9
- U1 pad 44: GPIO10 -> GPIO8
- U1 pad 45: GPIO9 -> GPIO7
- U1 pad 46: GPIO8 -> GPIO6
- U1 pad 47: GPIO7 -> Net-(R16-Pad2)
- U1 pad 48: GPIO6 -> Net-(R15-Pad2)
- U12 pad 6: Net-(U12-Pad11) -> Net-(R7-Pad1)
- U23 pad 6: Net-(U23-Pad11) -> Net-(R14-Pad2)
Routing:
- net Net-(J3-Pad1): track 0.00 -> 78.9 mm
- net Net-(J2-Pad1): track 0.00 -> 62.1 mm
- net Net-(R16-Pad2): track 0.00 -> 45.3 mm, vias 0 -> 1
- net Net-(R15-Pad2): track 0.00 -> 35.3 mm, vias 0 -> 1
- net Net-(U12-Pad11): track 5.40 -> 0.00 mm
- net Net-(U23-Pad11): track 5.40 -> 0.00 mm
- net Net-(D2-Pad2): track 0.00 -> 4.12 mm
- net Net-(D1-Pad2): track 0.00 -> 3.28 mm
- net +3V3: track 122.6 -> 125.2 mm
- net GPIO6: track 84.0 -> 86.5 mm
- net GPIO8: track 79.8 -> 82.2 mm
- net GPIO9: track 77.7 -> 80.0 mm
- net GPIO7: track 81.9 -> 84.0 mm
- net GPIO11: track 71.5 -> 73.6 mm
- net GPIO10: track 75.4 -> 77.5 mm
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
Commit message: merged in benchmarking into v3b. changed 3.3v power pin so that design is compatible with teensy 3.1/2 and 3.5/6.
Connections:
- U1 pad 15: +3V3 -> Net-(U1-Pad15)
- U1 pad 51: Net-(U1-Pad51) -> +3V3
Routing:
- net +3V3: track 125.2 -> 171.9 mm, vias 7 -> 9
