File: PCBs/MainPCB/microstim.sch (KiCad schematic (older format))
At the start: 87 parts, among them J1 Conn_Coaxial, J10 Conn_Coaxial, J11 Screw_Terminal_01x02, J12 Conn_Coaxial, J3 Screw_Terminal_01x02, J5 Conn_Coaxial, J7 Screw_Terminal_01x02, J9 Screw_Terminal_01x02, U1 Teensy3.5, U10 AD7321, U11 INA826, U12 AD8276, U13 AD8276, U14 INA826, U15 OPA197, U16 DG509ACWE, U17 OPA197, U18 DG509ACWE, U19 DG419LDY, U2 CC3-0512DF-E, U20 DG419LDY, U3 L78L05_SO8, U4 L78L12_SO8, U5 ISO7760, U6 AD1582, U7 ISO7341C, U8 L79L12_SO8, U9 MCP4922

Commit message: almost done with revision 3. 12v regs removed, GPIO breakout and indicator LEDs added, layout cleaned up
Parts:
- removed C14, C6: 1uF, Capacitor_SMD:C_0603_1608Metric, symbol Device:C_Small
- removed R10, R12: 100, Resistor_SMD:R_0603_1608Metric, symbol Device:R_US
- removed R11, R14: 180, Resistor_SMD:R_0603_1608Metric, symbol Device:R_US
- removed U4: L78L12_SO8, Package_SO:SOIC-8_3.9x4.9mm_P1.27mm, symbol Regulator_Linear:L78L12_SO8
- removed U8: L79L12_SO8, Package_SO:SOIC-8_3.9x4.9mm_P1.27mm, symbol Regulator_Linear:L79L12_SO8
- removed U9: MCP4922, Package_SO:SOIC-14_3.9x8.7mm_P1.27mm, symbol Analog_DAC:MCP4922
- added D1, D2: LED, LED_THT:LED_D5.0mm_Horizontal_O1.27mm_Z3.0mm, symbol Device:LED
- added J2: Conn_02x08_Counter_Clockwise, Connector_Multicomp:Multicomp_MC9A22-1634_2x08_P2.54mm_Horizontal, symbol Connector_Generic:Conn_02x08_Counter_Clockwise
- added SW1: SW_Push, Button_Switch_SMD:SW_SPST_EVPBF, symbol Switch:SW_Push
- added U4: AD5752, Package_SO:TSSOP-24_4.4x7.8mm_P0.65mm, symbol natecermak:AD5752
- C4, C8: value 1uF -> 0.1uF
- R17, R18: value 4k -> 500
- R3, R6: value 250 -> 100
- R7, R8: value 1.2k -> 1.8k
Connections:
- net labels added: GPIO0, GPIO1, GPIO2, GPIO3, GPIO4, GPIO5
- net labels removed: +12V, -12V
- wire segments 385 -> 426
Other:
- note added: "Max current output (0ohm load) is 10V/3k = +- 3.33mA.\nCurrent resolution is 20V/2^16/3k = 0.1uA\nMax voltage output (infinite load) is 40/43*15V = +/-13.95V"
- note added: "gain is Rsense*(1+49.4k/Rg) = 100*(1+49.4k/1.8k) = 2.84 mV/uA\nVoltage output range is thus +-3333*0.00284 = +-9.48V\noutput needs to be within +-10V\ncurrent sensing resolution is 10000 mV / 2^12 / (2.84mV/uA) = 0.86uA\n\n"
- note removed: "Max current output (0ohm load) is 2.5V/3k = +- 833uA.\nCurrent resolution is 5V/4096/3k = 0.4uA\nMax voltage output (infinite load) is 40/43*12V = 11.16V"
- note removed: "gain is Rsense*(1+49.4k/Rg) = 250*(1+49.4k/1.2k) = 10.5 mV/uA\nVoltage output range is thus +-833*0.0105 = +-8.7V\noutput needs to be within +-10V\n"
- moved on the sheet: C1, C10, C11, C13, C15, C16, C17, C18, C19, C2, C20, C21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

Commit message: major updates to isolate each output channel.
Parts:
- removed U19, U20: DG419LDY, Package_SO:SOIC-8_3.9x4.9mm_P1.27mm, symbol Analog_Switch:DG419LDY
- added C14, C37, C38, C41, C44, C46, C47, C49, C50, C6: 0.1uF, Capacitor_SMD:C_0603_1608Metric, symbol Device:C_Small
- added C35: 10uF, Capacitor_SMD:C_1206_3216Metric_Pad1.42x1.75mm_HandSolder, symbol Device:C_Small
- added C39, C45, C48: 1uF, Capacitor_SMD:C_0603_1608Metric, symbol Device:C_Small
- added C43: 680nF, Capacitor_SMD:C_0603_1608Metric, symbol Device:C_Small
- added U19: ISO7341C, Package_SO:SOIC-16W_7.5x10.3mm_P1.27mm, symbol Isolator:ISO7341C
- added U20: L78L05_SO8, Package_SO:SOIC-8_3.9x4.9mm_P1.27mm, symbol Regulator_Linear:L78L05_SO8
- added U21: AD5752, Package_SO:TSSOP-24_4.4x7.8mm_P0.65mm, symbol natecermak:AD5752
- added U22: AD7321, Package_SO:TSSOP-14_4.4x5mm_P0.65mm, symbol natecermak:AD7321
- added U23: AD1582, Package_TO_SOT_SMD:SOT-23, symbol natecermak:AD1582
- added U8: CC3-0512DF-E, microstim:CC3-0512DF-E, symbol natecermak:CC3-0512DF-E
- added U9: ISO7760, Package_SO:SOIC-16W_7.5x10.3mm_P1.27mm, symbol natecermak:ISO7760
- C32, C34: value 0.1uF -> 10uF; footprint Capacitor_SMD:C_0603_1608Metric -> Capacitor_SMD:C_1206_3216Metric_Pad1.42x1.75mm_HandSolder
Connections:
- net labels added: +15V_0, +15V_1, +5V_0, +5V_1, -15V_0, -15V_1, 2.5V_0, 2.5V_1, CS0_0, CS0_0i, CS0_1, CS0_1i, CS1_0, CS1_0i, CS1_1, CS1_1i, DAC_0, DAC_1, GND_0, GND_1, IOUT_0, IOUT_1, ISENSE_0, ISENSE_1, MISO_0, MISO_0i, MISO_1, MISO_1i, MOSI_0, MOSI_0i, MOSI_1, MOSI_1i, NLDAC_0, NLDAC_0i, NLDAC_1, NLDAC_1i, OE0_0, OE0_0i, OE0_1, OE0_1i, OE1_0, OE1_0i, OE1_1, OE1_1i, OUT_0, OUT_1, SCK_0, SCK_0i, SCK_1, SCK_1i, VOUT_0, VOUT_1
- net labels removed: 2.5V, CS0, CS0i, CS1, CS1i, DAC0, DAC1, IOUT0, IOUT1, ISENSE0, ISENSE1, MISO, MISOi, MOSI, MOSIi, NLDAC, NLDACi, OE0, OE0i, OE1, OE1i, OE2, OE2i, OE3, OE3i, OUT0, OUT1, SCK0, SCK0i, VOUT0, VOUT1
- wire segments 426 -> 535
Other:
- moved on the sheet: C1, C10, C11, C12, C13, C15, C16, C17, C18, C19, C2, C20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

Commit message: making progress on layout... slowly
Parts:
- added C51, C?: 1uF, Capacitor_SMD:C_0603_1608Metric, symbol Device:C_Small
- renumbered C3 to C1, C42 to C10, C4 to C11, C7 to C12, C8 to C13, C15 to C14, C12 to C15, C27 to C18, C21 to C19, C5 to C2, C28 to C20, C20 to C21, C36 to C22, C31 to C23, C33 to C24, C40 to C25, C6 to C26, C14 to C27, C32 to C28, C34 to C29, C1 to C3, C35 to C30, C37 to C31, C38 to C32, C39 to C33, C41 to C34, C44 to C35, C43 to C36, C45 to C37, C46 to C38, C47 to C39, C10 to C4, C48 to C40, C49 to C41, C50 to C42, C29 to C43, C30 to C44, C18 to C45, C19 to C46, C24 to C47, C22 to C48, C23 to C49, C26 to C5, C25 to C50, C11 to C6, C9 to C7, C2 to C8, C13 to C9, J2 to J1, J5 to J2, J1 to J3, J7 to J4, J3 to J5, J9 to J6, J10 to J7, J11 to J8, J12 to J9, R15 to R1, R18 to R10, R4 to R11, R6 to R12, R8 to R13, R9 to R14, R1 to R2, R17 to R3, R5 to R4, R3 to R5, R7 to R6, R13 to R7, R16 to R8, R2 to R9, U12 to U10, U18 to U12, U8 to U13, U9 to U14, U19 to U15, U20 to U16, U21 to U17, U22 to U18, U23 to U19, U17 to U20, U13 to U21, U14 to U22, U16 to U23, U5 to U3, U7 to U4, U3 to U5, U4 to U6, U10 to U7, U6 to U8, U15 to U9
Connections:
- net +15V is gone; now on net +15V_0: C18.2, C19.2, C23.2, C25.2, U10.7 (V+), U11.8 (+Vs), U12.14 (V+), U9.7 (V+)
- net +5V is gone; now on net +5V_0: U12.2 (EN)
- net -15V is gone; now on net -15V_0: C20.1, C21.1, C22.2, C24.2, U10.4 (V-), U11.5 (-Vs), U12.3 (V-), U9.4 (V-)
- net GNDREF is gone; now on net GND_0: C18.1, C20.2, C22.1, C23.1, C24.1, C25.1, J6.2 (Pin_2), J7.2 (Ext), R7.2, U11.6 (REF), U12.10 (S4B), U12.15 (GND)
- net +5V_0: now also C51.2
- net +5V_1: now also C?.2
- net GND: no longer U1.50 (23_A9_PWM_Touch)
- net GND_0: now also C51.1
- net GND_1: now also C?.1
- net at J2.1 (In), J4.1 (Pin_1): now also U1.50 (23_A9_PWM_Touch)
- net MISO_0 renamed MISO
- net MISO: now also U15.6 (OUTD)
- net MISO_1: no longer names the net of U1.3 (1_TX1_MISO1_Touch)
- net MISO_1: no longer U15.6 (OUTD)
- net MOSI_0 renamed MOSI
- net MOSI: now also U15.3 (INA)
- net MOSI_1: no longer names the net of U1.2 (0_RX1_MOSI1_Touch)
- net MOSI_1: no longer U15.3 (INA)
- net SCK_0 renamed SCK
- net SCK: now also U15.4 (INB)
- net SCK_1: no longer names the net of U1.24 (32_A13_TX4_SCK1)
- net SCK_1: no longer U15.4 (INB)
Other:
- moved on the sheet: C26, C27, C28, C29, C30, C31, C32, C33, C34, C35, C36, C37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

Commit message: getting darn close to done with layout.
Parts:
- removed J1: Conn_02x08_Counter_Clockwise, Connector_Multicomp:Multicomp_MC9A22-1634_2x08_P2.54mm_Horizontal, symbol Connector_Generic:Conn_02x08_Counter_Clockwise
- added J1: Conn_02x08_Odd_Even, Connector_Multicomp:Multicomp_MC9A22-1634_2x08_P2.54mm_Horizontal, symbol Connector_Generic:Conn_02x08_Odd_Even
- gave numbers to parts that had none: 1
Connections:
- net +3V3: now also U1.26 (3.3V), J1.1 (Pin_1)
- net CS0_0: now also U1.11 (9_PWM_RX2_CS0); no longer U1.12 (10_PWM_TX2_CS0)
- net CS0_1: now also U1.6 (4_PWM_CAN0RX_SDA2); no longer U1.7 (5_PWM_tx1_miso1)
- net CS1_0: now also U1.10 (8_TX3_miso0_sda0); no longer U1.11 (9_PWM_RX2_CS0)
- net CS1_1: now also U1.5 (3_PWM_CAN0TX_SCL2); no longer U1.6 (4_PWM_CAN0RX_SDA2)
- net GND: now also J1.3 (Pin_3), J1.4 (Pin_4)
- net GPIO0: now also U1.33 (36_A17_PWM), J1.5 (Pin_5); no longer U1.48 (21_A7_PWM_CS0_sck1)
- net GPIO1: now also U1.34 (37_A18_PWM_SCL1), J1.7 (Pin_7); no longer U1.47 (20_A6_PWM_CS0_sck1)
- net GPIO2: now also U1.35 (38_A19_PWM_SDA1), J1.9 (Pin_9); no longer U1.46 (19_A5_SCL0_Touch)
- net GPIO3: now also U1.36 (39_A20), J1.11 (Pin_11); no longer U1.45 (18_A4_SDA0_Touch)
- net GPIO4: now also U1.37 (A21_DAC0), J1.13 (Pin_13); no longer U1.44 (17_A3_sda0_Touch)
- net GPIO5: now also U1.38 (A22_DAC1), J1.15 (Pin_15); no longer U1.43 (16_A2_scl0_Touch)
- net NLDAC_0: now also U1.12 (10_PWM_TX2_CS0); no longer U1.16 (24)
- net NLDAC_1: now also U1.7 (5_PWM_tx1_miso1); no longer U1.8 (6_PWM)
- net OE0_0: now also U1.9 (7_RX3_miso0_scl0); no longer U1.10 (8_TX3_miso0_sda0)
- net OE0_1: now also U1.4 (2_PWM); no longer U1.5 (3_PWM_CAN0TX_SCL2)
- net OE1_0: now also U1.8 (6_PWM); no longer U1.9 (7_RX3_miso0_scl0)
- net OE1_1: now also U1.3 (1_TX1_MISO1_Touch); no longer U1.4 (2_PWM)
- net VUSB: now also J1.2 (Pin_2)
- new net GPIO10: J1.14 (Pin_14), U1.44 (17_A3_sda0_Touch)
- new net GPIO11: J1.16 (Pin_16), U1.43 (16_A2_scl0_Touch)
- new net GPIO6: J1.6 (Pin_6), U1.48 (21_A7_PWM_CS0_sck1)
- new net GPIO7: J1.8 (Pin_8), U1.47 (20_A6_PWM_CS0_sck1)
- new net GPIO8: J1.10 (Pin_10), U1.46 (19_A5_SCL0_Touch)
- new net GPIO9: J1.12 (Pin_12), U1.45 (18_A4_SDA0_Touch)
Changed lines of the file:
@@
 Text GLabel 7350 1900 0    50   Input ~ 0
 OE0_0
-Text GLabel 1800 3150 0    50   Input ~ 0
+Text GLabel 1800 2750 0    50   Input ~ 0
 NLDAC_0
 $Comp
@@
 Wire Wire Line
 	8250 2350 8500 2350
-Text GLabel 1800 2650 0    50   Input ~ 0
+Text GLabel 1800 2550 0    50   Input ~ 0
 CS1_0
-Text GLabel 1800 2750 0    50   Input ~ 0
+Text GLabel 1800 2650 0    50   Input ~ 0
 CS0_0
 Wire Wire Line
@@
 Wire Wire Line
 	16750 4850 16900 4850
-Text GLabel 1800 2450 0    50   Input ~ 0
+Text GLabel 1800 2350 0    50   Input ~ 0
 OE1_0
-Text GLabel 1800 2550 0    50   Input ~ 0
+Text GLabel 1800 2450 0    50   Input ~ 0
 OE0_0
 Wire Wire Line
@@
 Wire Wire Line
 	1850 4350 1950 4350
-$Comp
-L Connector_Generic:Conn_02x08_Counter_Clockwise J1
-U 1 1 5CBED068
-P 900 5050
-F 0 "J1" H 950 4517 50  0000 C CNN
-F 1 "Conn_02x08_Counter_Clockwise" H 950 4426 50  0000 C CNN
-F 2 "Connector_Multicomp:Multicomp_MC9A22-1634_2x08_P2.54mm_Horizontal" H 900 5050 50  0001 C CNN
-F 3 "~" H 900 5050 50  0001 C CNN
-	1    900  5050
-	1    0    0    -1
-$EndComp
-Wire Wire Line
-	700  4250 700  4750
-Wire Wire Line
-	700  4850 600  4850
-Wire Wire Line
-	600  4850 600  4150
 Wire Wire Line
-	500  4950 700  4950
+	5000 3600 5100 3600
 Wire Wire Line
-	500  5050 700  5050
+	5000 3700 5100 3700
 Wire Wire Line
-	500  5150 700  5150
+	5000 3800 5100 3800
 Wire Wire Line
-	500  5250 700  5250
+	5000 3900 5100 3900
 Wire Wire Line
-	500  5350 700  5350
+	5000 4000 5100 4000
 Wire Wire Line
-	700  5450 500  5450
-Wire Wire Line
-	1950 5350 1200 5350
-Wire Wire Line
-	1200 5250 1950 5250
+	5100 4100 5000 4100
 Wire Wire Line
 	9950 150  10500 150
@@
 	1    0    0    -1
 $EndComp
-$Comp
-L power:GND #PWR01
-U 1 1 5C5D1E51
-P 850 4250
-F 0 "#PWR01" H 850 4000 50  0001 C CNN
-F 1 "GND" H 855 4077 50  0000 C CNN
-F 2 "" H 850 4250 50  0001 C CNN
-F 3 "" H 850 4250 50  0001 C CNN
-	1    850  4250
-	1    0    0    -1
-$EndComp
-Wire Wire Line
-	700  4250 850  4250
 Wire Wire Line
 	1950 4250 1400 4250
@@
 	1400 4350 1400 4450
 Wire Wire Line
-	1950 5050 1700 5050
-Wire Wire Line
-	1700 5050 1700 5150
-Wire Wire Line
-	1700 5150 1200 5150
-Wire Wire Line
-	1200 5050 1600 5050
-Wire Wire Line
-	1600 5050 1600 4950
-Wire Wire Line
-	1600 4950 1950 4950
-Wire Wire Line
-	1200 4950 1500 4950
-Wire Wire Line
-	1500 4950 1500 4850
-Wire Wire Line
-	1500 4850 1950 4850
-Wire Wire Line
-	1200 4850 1400 4850
-Wire Wire Line
-	1400 4850 1400 4750
-Wire Wire Line
-	1950 4750 1400 4750
-Wire Wire Line
-	1200 4750 1300 4750
-Wire Wire Line
-	1300 4750 1300 4150
-Wire Wire Line
 	1300 4150 1950 4150
-Text GLabel 600  4150 2    50   Input ~ 0
+Text GLabel 5700 3400 2    50   Input ~ 0
 VUSB
-Wire Wire Line
-	1200 5450 1400 5450
 $Comp
 L power:GND #PWR05
 U 1 1 5C9B26A7
-P 1400 5450
-F 0 "#PWR05" H 1400 5200 50  0001 C CNN
-F 1 "GND" H 1405 5277 50  0000 C CNN
-F 2 "" H 1400 5450 50  0001 C CNN
-F 3 "" H 1400 5450 50  0001 C CNN
-	1    1400 5450
-	1    0    0    -1
+P 4500 3500
+F 0 "#PWR05" H 4500 3250 50  0001 C CNN
+F 1 "GND" H 4505 3327 50  0000 C CNN
+F 2 "" H 4500 3500 50  0001 C CNN
+F 3 "" H 4500 3500 50  0001 C CNN
+	1    4500 3500
+	-1   0    0    -1
 $EndComp
-Connection ~ 1400 5450
-Wire Wire Line
-	1400 5450 1950 5450
-Text GLabel 500  5450 0    50   Input ~ 0
+Text GLabel 5000 4100 0    50   Input ~ 0
 GPIO5
-Text GLabel 500  5350 0    50   Input ~ 0
+Text GLabel 5000 4000 0    50   Input ~ 0
 GPIO4
-Text GLabel 500  5250 0    50   Input ~ 0
+Text GLabel 5000 3900 0    50   Input ~ 0
 GPIO3
-Text GLabel 500  5050 0    50   Input ~ 0
+Text GLabel 5000 3700 0    50   Input ~ 0
 GPIO1
-Text GLabel 500  5150 0    50   Input ~ 0
+Text GLabel 5000 3800 0    50   Input ~ 0
 GPIO2
-Text GLabel 500  4950 0    50   Input ~ 0
+Text GLabel 5000 3600 0    50   Input ~ 0
 GPIO0
-Text GLabel 1750 5850 0    50   Input ~ 0
+Text GLabel 1750 5350 0    50   Input ~ 0
 GPIO5
-Text GLabel 4100 5850 2    50   Input ~ 0
+Text GLabel 1800 5250 0    50   Input ~ 0
 GPIO4
-Text GLabel 4100 5750 2    50   Input ~ 0
+Text GLabel 1800 5150 0    50   Input ~ 0
 GPIO3
-Text GLabel 4100 5550 2    50   Input ~ 0
+Text GLabel 1800 4950 0    50   Input ~ 0
 GPIO1
-Text GLabel 4100 5650 2    50   Input ~ 0
+Text GLabel 1800 5050 0    50   Input ~ 0
 GPIO2
-Text GLabel 4100 5450 2    50   Input ~ 0
+Text GLabel 1800 4850 0    50   Input ~ 0
 GPIO0
 Wire Wire Line
-	1750 5850 1950 5850
+	1750 5350 1950 5350
 Wire Wire Line
-	3950 5850 4100 5850
+	1950 5250 1800 5250
 Wire Wire Line
-	4100 5750 3950 5750
+	1800 5150 1950 5150
 Wire Wire Line
-	3950 5650 4100 5650
+	1950 5050 1800 5050
 Wire Wire Line
-	4100 5550 3950 5550
+	1800 4950 1950 4950
 Wire Wire Line
-	3950 5450 4100 5450
-Text GLabel 1800 2350 0    50   Input ~ 0
-NLDAC_1
+	1950 4850 1800 4850
 Text GLabel 1800 2250 0    50   Input ~ 0
-CS0_1
+NLDAC_1
 Text GLabel 1800 2150 0    50   Input ~ 0
+CS0_1
+Text GLabel 1800 2050 0    50   Input ~ 0
 CS1_1
-Text GLabel 1800 1950 0    50   Input ~ 0
+Text GLabel 1800 1850 0    50   Input ~ 0
 OE1_1
-Text GLabel 1800 2050 0    50   Input ~ 0
+Text GLabel 1800 1950 0    50   Input ~ 0
 OE0_1
 Wire Wire Line
-	1800 2350 1950 2350
-Wire Wire Line
 	1800 2250 1950 2250
 Wire Wire Line
 	1800 2150 1950 2150
 Wire Wire Line
-	1800 1950 1950 1950
-Wire Wire Line
 	1800 2050 1950 2050
 Wire Wire Line
-	1800 3150 1950 3150
+	1800 1850 1950 1850
 Wire Wire Line
-	1800 2750 1950 2750
+	1800 1950 1950 1950
 Wire Wire Line
-	1950 2650 1800 2650
+	1800 2650 1950 2650
 Wire Wire Line
-	1800 2550 1950 2550
+	1950 2550 1800 2550
 Wire Wire Line
-	1950 2450 1800 2450
+	1800 2450 1950 2450
+Wire Wire Line
+	1950 2350 1800 2350
 Wire Wire Line
 	10750 3850 10900 3850
@@
 	10500 450  10950 450
 $Comp
-L Device:C_Small C?
+L Device:C_Small C52
 U 1 1 5C9B5470
 P 10650 5100
-F 0 "C?" H 10558 5054 50  0000 R CNN
+F 0 "C52" H 10558 5054 50  0000 R CNN
 F 1 "1uF" H 10558 5145 50  0000 R CNN
 F 2 "Capacitor_SMD:C_0603_1608Metric" H 10650 5100 50  0001 C CNN
@@
 Wire Wire Line
 	10650 5300 11100 5300
+Wire Wire Line
+	1800 2750 1950 2750
+Text GLabel 5700 4000 2    50   Input ~ 0
+GPIO10
+Text GLabel 5700 3900 2    50   Input ~ 0
+GPIO9
+Text GLabel 5700 3700 2    50   Input ~ 0
+GPIO7
+Text GLabel 5700 3800 2    50   Input ~ 0
+GPIO8
+Text GLabel 5700 3600 2    50   Input ~ 0
+GPIO6
+$Comp
+L power:GND #PWR0110
+U 1 1 5CC7B82D
+P 1550 5450
+F 0 "#PWR0110" H 1550 5200 50  0001 C CNN
+F 1 "GND" H 1555 5277 50  0000 C CNN
+F 2 "" H 1550 5450 50  0001 C CNN
+F 3 "" H 1550 5450 50  0001 C CNN
+	1    1550 5450
+	1    0    0    -1
+$EndComp
+Wire Wire Line
+	1550 5450 1950 5450
+Wire Wire Line
+	5700 3400 5600 3400
+$Comp
+L power:+3.3V #PWR0111
+U 1 1 5D1270A2
+P 1300 4150
+F 0 "#PWR0111" H 1300 4000 50  0001 C CNN
+F 1 "+3.3V" H 1315 4323 50  0000 C CNN
+F 2 "" H 1300 4150 50  0001 C CNN
+F 3 "" H 1300 4150 50  0001 C CNN
+	1    1300 4150
+	1    0    0    -1
+$EndComp
+Text GLabel 5700 4100 2    50   Input ~ 0
+GPIO11
+Wire Wire Line
+	5600 4100 5700 4100
+Wire Wire Line
+	5600 4000 5700 4000
+Wire Wire Line
+	5600 3900 5700 3900
+Wire Wire Line
+	5600 3800 5700 3800
+Wire Wire Line
+	5600 3700 5700 3700
+Wire Wire Line
+	5600 3600 5700 3600
+$Comp
+L power:+3.3V #PWR0112
+U 1 1 5D3D870A
+P 4800 3400
+F 0 "#PWR0112" H 4800 3250 50  0001 C CNN
+F 1 "+3.3V" H 4815 3573 50  0000 C CNN
+F 2 "" H 4800 3400 50  0001 C CNN
+F 3 "" H 4800 3400 50  0001 C CNN
+	1    4800 3400
+	-1   0    0    -1
+$EndComp
+Text GLabel 4050 5850 2    50   Input ~ 0
+GPIO10
+Text GLabel 4050 5750 2    50   Input ~ 0
+GPIO9
+Text GLabel 4050 5550 2    50   Input ~ 0
+GPIO7
+Text GLabel 4050 5650 2    50   Input ~ 0
+GPIO8
+Text GLabel 4050 5450 2    50   Input ~ 0
+GPIO6
+Text GLabel 1850 5850 0    50   Input ~ 0
+GPIO11
+Wire Wire Line
+	4050 5450 3950 5450
+Wire Wire Line
+	4050 5550 3950 5550
+Wire Wire Line
+	4050 5650 3950 5650
+Wire Wire Line
+	4050 5750 3950 5750
+Wire Wire Line
+	4050 5850 3950 5850
+Wire Wire Line
+	1850 5850 1950 5850
+Wire Wire Line
+	4800 3400 5100 3400
+$Comp
+L Connector_Generic:Conn_02x08_Odd_Even J1
+U 1 1 5DFCF206
+P 5300 3700
+F 0 "J1" H 5350 4217 50  0000 C CNN
+F 1 "Conn_02x08_Odd_Even" H 5350 4126 50  0000 C CNN
+F 2 "Connector_Multicomp:Multicomp_MC9A22-1634_2x08_P2.54mm_Horizontal" H 5300 3700 50  0001 C CNN
+F 3 "~" H 5300 3700 50  0001 C CNN
+	1    5300 3700
+	1    0    0    -1
+$EndComp
+Wire Wire Line
+	4500 3500 5100 3500
+$Comp
+L power:GND #PWR0113
+U 1 1 5E353902
+P 6100 3500
+F 0 "#PWR0113" H 6100 3250 50  0001 C CNN
+F 1 "GND" H 6105 3327 50  0000 C CNN
+F 2 "" H 6100 3500 50  0001 C CNN
+F 3 "" H 6100 3500 50  0001 C CNN
+	1    6100 3500
+	-1   0    0    -1
+$EndComp
+Wire Wire Line
+	5600 3500 6100 3500
 $EndSCHEMATC

Commit message: finished layout, schematic+pcb pdfs, BOM. need to do panels.
Parts:
- removed J4, J5: Screw_Terminal_01x02, microstim:1-2834016-2 _TERM_BLK_2P_SIDE_ENT_2.54MM_PCB, symbol Connector:Screw_Terminal_01x02
- added R15, R16: 200, Resistor_SMD:R_0603_1608Metric, symbol Device:R_US
- D1, D2: footprint LED_THT:LED_D5.0mm_Horizontal_O1.27mm_Z3.0mm -> microstim:LED_D5.0mm_Horizontal_O1.27mm_Z3.0mm_pinSwapped
- SW1: footprint Button_Switch_SMD:SW_SPST_EVPBF -> microstim:EVQ-PF303K
Connections:
- net +3V3: now also J1.3 (Pin_3); no longer J1.1 (Pin_1)
- net GND: now also D1.1 (K), D2.1 (K), J1.1 (Pin_1); no longer J1.3 (Pin_3)
- net GPIO10: now also U1.42 (15_A1_CS0_Touch); no longer U1.44 (17_A3_sda0_Touch)
- net GPIO11: now also U1.41 (14_A0_PWM_sck0); no longer U1.43 (16_A2_scl0_Touch)
- net GPIO6: now also U1.46 (19_A5_SCL0_Touch); no longer U1.48 (21_A7_PWM_CS0_sck1)
- net GPIO7: now also U1.45 (18_A4_SDA0_Touch); no longer U1.47 (20_A6_PWM_CS0_sck1)
- net GPIO8: now also U1.44 (17_A3_sda0_Touch); no longer U1.46 (19_A5_SCL0_Touch)
- net GPIO9: now also U1.43 (16_A2_scl0_Touch); no longer U1.45 (18_A4_SDA0_Touch)
- net at U12.11 (S3B): no longer U12.6 (S3A)
- net at R7.1, U12.4 (S1A), U12.7 (S4A): now also U12.6 (S3A)
- net at U23.11 (S3B): no longer U23.6 (S3A)
- net at R14.2, U23.4 (S1A), U23.7 (S4A): now also U23.6 (S3A)
- net at D1.2 (A): now also R15.1
- net at D2.2 (A): now also R16.1
- new net: R16.2, U1.47 (20_A6_PWM_CS0_sck1)
- new net: R15.2, U1.48 (21_A7_PWM_CS0_sck1)
Other:
- note added: "Max current output (0ohm load) is (+/-10V)/3k = +- 3.33mA.\nCurrent resolution is 20V/2^16/3k = 0.1uA\nMax voltage output (infinite load) is 40/43*14.8V = +/-13.76V"
- note added: "OE0 OE1 Output \n\n 0 0 VOLTAGE \n 1 0 CURRENT \n 0 1 High-Z \n 1 1 GND"
- note added: "Stim channel 0"
- note added: "Stim channel 1"
- note added: "gain is Rsense*(1+49.4k/Rg) = 100*(1+49.4k/1.8k) = 2.87 mV/uA\nVoltage output range is thus +-3333*0.00287 = +-9.57V\noutput needs to be within +-10V\ncurrent sensing resolution is 10000 mV / 2^12 / (2.87mV/uA) = 0.85uA\n\n"
- note removed: "Max current output (0ohm load) is 10V/3k = +- 3.33mA.\nCurrent resolution is 20V/2^16/3k = 0.1uA\nMax voltage output (infinite load) is 40/43*15V = +/-13.95V"
- note removed: "OE0 OE1 Output Input (ADC)\n\n 0 0 VOLTAGE OUT0\n 1 0 CURRENT OUT0\n 0 1 CURRENT ISENSE0\n 1 1 GND ISENSE0"
- note removed: "gain is Rsense*(1+49.4k/Rg) = 100*(1+49.4k/1.8k) = 2.84 mV/uA\nVoltage output range is thus +-3333*0.00284 = +-9.48V\noutput needs to be within +-10V\ncurrent sensing resolution is 10000 mV / 2^12 / (2.84mV/uA) = 0.86uA\n\n"
- moved on the sheet: C1, C10, C11, C12, C13, C14, C15, C16, C17, C18, C19, C2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
