File: PCB/stimjim_pcb_kicad/mcu.kicad_sch (KiCad schematic)
At the start: 41 parts, among them J2 Conn_Coaxial, J3 Conn_Coaxial, SW2 PTS645VH58-2 LFS, SW3 TS04-66-50-BK-160-SMT, U24 RP2354B, U25 W25Q128JVS, Y1 ABM8AIG-12.000MHZ-12-2Z-T3

Commit message: Simplified layout
- Went to 4 layers
- Simplified GPIO interface and remove power connections since they are
  a recipe for disaster
- Independent SPI busses to each stimulator to allow simultaneous
  control
Parts:
- removed C63, C65: 100n, Capacitor_SMD:C_0402_1005Metric, symbol Device:C
- removed R16: 0, Resistor_SMD:R_0402_1005Metric, symbol Device:R_US
- C55, C56, C57, C58, C59, C60, C61, C62, C64, C81, C83, C84: value 100n -> 0.1uF
- U24: footprint Package_DFN_QFN:QFN-80-1EP_10x10mm_P0.4mm_EP3.4x3.4mm -> Package_DFN_QFN:QFN-80-1EP_10x10mm_P0.4mm_EP3.4x3.4mm_ThermalVias
Connections:
- net FLASH_SS is gone; now on net ~{QSPI_SS}: U25.1 (~{CS})
- net GPIO10 is gone; now on net GPIO7: U24.8 (GPIO10)
- net GPIO11 is gone; now on net GPIO1: U24.12 (GPIO13)
- net GPIO8 is gone; now on net GPIO4: U24.3 (GPIO6)
- net GPIO9 is gone; now on net GPIO6: U24.7 (GPIO9)
- net OE1_0 is gone; now on an unnamed net: U24.42 (GPIO33)
- net GPIO0: now also U24.13 (GPIO14); no longer U24.21 (GPIO21)
- net GPIO1: no longer U24.20 (GPIO20)
- net GPIO2: now also U24.1 (GPIO4); no longer U24.19 (GPIO19)
- net GPIO3: now also U24.2 (GPIO5); no longer U24.18 (GPIO18)
- net GPIO4: no longer U24.17 (GPIO17)
- net GPIO5: now also U24.4 (GPIO7); no longer U24.13 (GPIO14)
- net GPIO6: no longer U24.1 (GPIO4)
- net GPIO7: no longer U24.2 (GPIO5)
- net at J2.1 (In): no longer U24.38 (GPIO30)
- net USB_D+: now reaches R31.1, U24.67 (USB_DP)
- net NLDAC_{B}: now reaches U24.25 (GPIO24)
- net at U24.39 (GPIO31): no longer J3.1 (In)
- net CSB_{A}: now reaches U24.52 (GPIO41/ADC1)
- net USB_D-: now reaches R30.1, U24.66 (USB_DM)
- net CS0_0 renamed OE1_{A}
- net CS0_1 renamed SCK_{A}
- net CS1_0: no longer names the net of U24.45 (GPIO36)
- net CS1_1 renamed CSA_{A}
- net MISO_0: no longer names the net of U24.40 (GPIO32)
- net MISO_1: no longer names the net of U24.44 (GPIO35)
- net MOSI renamed MOSI_{B}
- net NLDAC_0 renamed OE0_{A}
- net NLDAC_1 renamed MOSI_{A}
- net OE0_0: no longer names the net of U24.43 (GPIO34)
- net OE0_0: now also J3.1 (In)
- net OE0_1 renamed MISO_{A}
- net OE1_1 renamed NLDAC_{A}
- net SCK renamed SCK_{B}
- new net CSA_{B}: U24.21 (GPIO21)
- new net CSB_{B}: U24.17 (GPIO17)
- new net MISO_{B}: U24.20 (GPIO20)
- new net OE0_{B}: U24.19 (GPIO19)
- new net OE1_{B}: U24.18 (GPIO18)
- no-connect marks 16 -> 18
Other:
- note added: "XX_{0} pertains to the SPI instance number."
- title: (none) -> StimJim
- moved on the sheet: C62, C64, J2, J3, R30, R31, U25

Commit message: filipe feedback
Parts:
- J2, J3: footprint microstim:731375003 -> Connector_Coaxial:BNC_Amphenol_B6252HB-NPP3G-50_Horizontal
Other:
- note added: "NB: Place resistors close to pins 66 & 67"
- note removed: "NB: Place resistors close to pins 46 & 47"
Changed lines of the file:
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@@
 		)
 	)
-	(text "NB: Place resistors\nclose to pins 46 & 47"
+	(text "NB: Place resistors\nclose to pins 66 & 67"
 		(exclude_from_sim no)
 		(at 93.98 137.16 0)
@@
 			)
 		)
-		(property "Footprint" "microstim:731375003"
+		(property "Footprint" "Connector_Coaxial:BNC_Amphenol_B6252HB-NPP3G-50_Horizontal"
 			(at 212.09 187.96 0)
 			(effects
@@
 			)
 		)
-		(property "Footprint" "microstim:731375003"
+		(property "Footprint" "Connector_Coaxial:BNC_Amphenol_B6252HB-NPP3G-50_Horizontal"
 			(at 189.23 190.5 0)
 			(effects
@@
 			)
 		)
-		(property "Datasheet" "~"
+		(property "Datasheet" "https://abracon.com/AIGcrystals/ABM8AIG.pdf"
 			(at 82.55 162.56 0)
 			(effects
