File: PCB/stimjim_pcb_kicad/panels.kicad_pcb (KiCad board)
At the start: 2 copper layers, 140 x 71 mm, 0 parts

Commit message: Merged in nc-update-to-kicad7 (pull request #3)
Update PCB design to kicad 7

* migrate to kicad7

* remove empty.kicad_wks; fix sheet size and add authors and version to page

* migrate libraries to new format; fix incorrectly rescued symbols (+3.3V power flag and L78L05-SO8 regulator)

* slowly fixing all ERC errors; down to 3

* fix ina826 symbol (again). down to 0 ERC errors; 56 warnings

* fixed all ERC errors in schematic; pulled changes into PCB (probably some new net names, but nothing obviously broken)

* DRC errors/warnings all resolved
Other:
- net class Default removed
- net class thick removed

Commit message: filipe feedback
Other:
- outline, holes or cut-outs redrawn
- board text added: "GND GND GND GND GND GND GND GND"
- board text added: "GPIO 1 GPIO 2 GPIO 3 GPIO 4 GPIO 5 GPIO 6 GPIO 7 GPIO 8"
- board text added: "POWER"
- board text added: "revB"
- board text removed: "11 10 09 08 07 06 GND VUSB"
- board text removed: "GND +3.3V 00 01 02 03 04 05"
- board text removed: "v0.18"
