File: PCB/stimjim.kicad_pcb (KiCad board)
At the start: 4 copper layers, 129 x 79.5 mm, 236 parts, among them J1 302-R161, J10 USB4105-GF-A, J11 BM03B-SRSS-TB, J2 0731375003, J3 0731375003, J4 10129383-910002ALF, J7 0731375003, J9 0731375003, SW2 PTS645VH58-2 LFS, SW3 TS04-66-50-BK-160-SMT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

Commit message: tolerance resistors
Parts:
- R11, R9: value 1k -> 0
- R13, R6: value 1.8k -> 360
- U24, U29: value AD8421BRZ -> AD8421
- U30: footprint Package_DFN_QFN:QFN-80-1EP_10x10mm_P0.4mm_EP3.4x3.4mm_ThermalVias -> Package_DFN_QFN:QFN-80-1EP_10x10mm_P0.4mm_EP3.4x3.4mm
