File: PCB/stimjim.kicad_pcb (KiCad board)
At the start: 4 copper layers, 129 x 79.5 mm, 236 parts, among them J1 302-R161, J10 USB4105-GF-A, J11 BM03B-SRSS-TB, J2 0731375003, J3 0731375003, J4 10129383-910002ALF, J7 0731375003, J9 0731375003, SW2 PTS645VH58-2 LFS, SW3 TS04-66-50-BK-160-SMT, U1 OPA197, U10 OPA197, U12 DG409DYZ-T, U13 CC3-0512DF-E, U14 ISO7760, U15 ISO7741, U151 AP2112K-3.3, U16 MC78L05ACDR2G, U17 AD5752, U18 AD7321, U19 AD1582, U2 CC3-0512DF-E, U20 OPA197, U21 OPA197, U23 DG409DYZ-T, U24 AD8421, U25 W25Q128JVS, U26 OPA197, U27 LT1995, U28 LT1995, U29 AD8421, U3 ISO7760, U30 RP2354B, U4 ISO7741, U5 MC78L05ACDR2G, U6 AD5752, U7 AD7321, U8 AD1582, U9 OPA197, Y1 ABM8AIG-12.000MHZ-12-2Z-T3

Commit message: Add ground connections to rp2354 thermal pad
- It was floating
- Fix some silkscreen issues
Routing:
- net GND: vias 115 -> 123
Changed lines of the file:
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@@
 		(grid_origin 147 168)
 		(pcbplotparams
-			(layerselection 0x00000000_00000000_5555555f_5755f5ff)
+			(layerselection 0x00000000_00000000_55555555_55555520)
 			(plot_on_all_layers_selection 0x00000000_00000000_00000000_00000000)
 			(disableapertmacros no)
@@
 			(at 0 1.43 90)
 			(layer "F.Fab")
+			(hide yes)
 			(effects
 				(font
@@
 			(at 0 1.43 0)
 			(layer "F.Fab")
+			(hide yes)
 			(effects
 				(font
@@
 			(at 0 1.43 0)
 			(layer "F.Fab")
+			(hide yes)
 			(effects
 				(font
@@
 			(at 0 1.43 90)
 			(layer "F.Fab")
+			(hide yes)
 			(effects
 				(font
@@
 			(at 0 1.43 90)
 			(layer "F.Fab")
+			(hide yes)
 			(effects
 				(font
@@
 			(at 0 2.45 0)
 			(layer "F.Fab")
+			(hide yes)
 			(effects
 				(font
@@
 			(at 0 1.43 90)
 			(layer "F.Fab")
+			(hide yes)
 			(effects
 				(font
@@
 			(at 0 2.45 0)
 			(layer "F.Fab")
+			(hide yes)
 			(effects
 				(font
@@
 			(at 0 1.43 90)
 			(layer "F.Fab")
+			(hide yes)
 			(effects
 				(font
@@
 			(at 0 -3.4 0)
 			(layer "F.Fab")
+			(hide yes)
 			(effects
 				(font
@@
 			(unlocked yes)
 			(layer "F.Fab")
+			(hide yes)
 			(effects
 				(font
@@
 			(at 0 1.43 0)
 			(layer "F.Fab")
+			(hide yes)
 			(effects
 				(font
@@
 			(at 0 1.43 90)
 			(layer "F.Fab")
+			(hide yes)
 			(effects
 				(font
@@
 			(at 6.215 23.88 90)
 			(layer "F.Fab")
+			(hide yes)
 			(effects
 				(font
@@
 			(at 0 1.43 0)
 			(layer "F.Fab")
+			(hide yes)
 			(effects
 				(font
@@
 			(at 0 3.4 0)
 			(layer "F.Fab")
+			(hide yes)
 			(effects
 				(font
@@
 			(at 0 1.43 0)
 			(layer "F.Fab")
+			(hide yes)
 			(effects
 				(font
@@
 			(at 0 1.43 0)
 			(layer "F.Fab")
+			(hide yes)
 			(effects
 				(font
@@
 			(at 0 1.43 0)
 			(layer "F.Fab")
+			(hide yes)
 			(effects
 				(font
@@
 			(at 0 3.4 0)
 			(layer "F.Fab")
+			(hide yes)
 			(effects
 				(font
@@
 			(at 0 1.43 90)
 			(layer "F.Fab")
+			(hide yes)
 			(effects
 				(font
@@
 			(at 0 1.43 0)
 			(layer "F.Fab")
+			(hide yes)
 			(effects
 				(font
@@
 			(unlocked yes)
 			(layer "F.Fab")
+			(hide yes)
 			(effects
 				(font
@@
 			(at 0 1.43 0)
 			(layer "F.Fab")
+			(hide yes)
 			(effects
 				(font
@@
 			(at 0 1.43 0)
 			(layer "F.Fab")
+			(hide yes)
 			(effects
 				(font
@@
 			(at 0 1.43 90)
 			(layer "F.Fab")
+			(hide yes)
 			(effects
 				(font
@@
 			(unlocked yes)
 			(layer "F.Fab")
+			(hide yes)
 			(effects
 				(font
@@
 			(at 0 1.43 0)
 			(layer "F.Fab")
+			(hide yes)
 			(effects
 				(font
@@
 			(at 0 1.43 0)
 			(layer "F.Fab")
+			(hide yes)
 			(effects
 				(font
@@
 			(at 0 -3.4 0)
 			(layer "F.Fab")
+			(hide yes)
 			(effects
 				(font
@@
 			(unlocked yes)
 			(layer "F.Fab")
+			(hide yes)
 			(effects
 				(font
@@
 			(at 0 1.43 90)
 			(layer "F.Fab")
+			(hide yes)
 			(effects
 				(font
@@
 			(at 0 1.43 90)
 			(layer "F.Fab")
+			(hide yes)
 			(effects
 				(font
@@
 		(tags "QFN NoLead")
 		(property "Reference" "U30"
-			(at 0 -6.3 180)
+			(at -6.725 -5.15 180)
 			(layer "F.SilkS")
 			(effects
@@
 			(at 0 6.3 180)
 			(layer "F.Fab")
+			(hide yes)
 			(effects
 				(font
@@
 	)
 	(via
+		(at 165 129.15)
+		(size 0.5)
+		(drill 0.3)
+		(layers "F.Cu" "B.Cu")
+		(free yes)
+		(capping no)
+		(covering
+			(front no)
+			(back no)
+		)
+		(plugging
+			(front no)
+			(back no)
+		)
+		(filling no)
+		(net "GND")
+	)
+	(via
 		(at 173.9 133.5)
 		(size 0.5)
@@
 	)
 	(via
+		(at 163.65 130.525)
+		(size 0.5)
+		(drill 0.3)
+		(layers "F.Cu" "B.Cu")
+		(free yes)
+		(capping no)
+		(covering
+			(front no)
+			(back no)
+		)
+		(plugging
+			(front no)
+			(back no)
+		)
+		(filling no)
+		(net "GND")
+	)
+	(via
 		(at 241.9 150.8)
 		(size 0.8)
@@
 	)
 	(via
+		(at 165.025 131.85)
+		(size 0.5)
+		(drill 0.3)
+		(layers "F.Cu" "B.Cu")
+		(free yes)
+		(capping no)
+		(covering
+			(front no)
+			(back no)
+		)
+		(plugging
+			(front no)
+			(back no)
+		)
+		(filling no)
+		(net "GND")
+	)
+	(via
 		(at 167.84125 115.3125)
 		(size 0.5)
@@
 	)
 	(via
+		(at 163.65 129.15)
+		(size 0.5)
+		(drill 0.3)
+		(layers "F.Cu" "B.Cu")
+		(free yes)
+		(capping no)
+		(covering
+			(front no)
+			(back no)
+		)
+		(plugging
+			(front no)
+			(back no)
+		)
+		(filling no)
+		(net "GND")
+	)
+	(via
 		(at 184.09125 123.8625)
 		(size 0.5)
@@
 	)
 	(via
-		(at 168.75 128)
+		(at 166.35 129.15)
 		(size 0.5)
 		(drill 0.3)
@@
 	)
 	(via
+		(at 166.35 131.85)
+		(size 0.5)
+		(drill 0.3)
+		(layers "F.Cu" "B.Cu")
+		(free yes)
+		(capping no)
+		(covering
+			(front no)
+			(back no)
+		)
+		(plugging
+			(front no)
+			(back no)
+		)
+		(filling no)
+		(net "GND")
+	)
+	(via
 		(at 157.24125 134.3125)
 		(size 0.5)
@@
 	)
 	(via
+		(at 166.35 130.5)
+		(size 0.5)
+		(drill 0.3)
+		(layers "F.Cu" "B.Cu")
+		(free yes)
+		(capping no)
+		(covering
+			(front no)
+			(back no)
+		)
+		(plugging
+			(front no)
+			(back no)
+		)
+		(filling no)
+		(net "GND")
+	)
+	(via
+		(at 163.65 131.85)
+		(size 0.5)
+		(drill 0.3)
+		(layers "F.Cu" "B.Cu")
+		(free yes)
+		(capping no)
+		(covering
+			(front no)
+			(back no)
+		)
+		(plugging
+			(front no)
+			(back no)
+		)
+		(filling no)
+		(net "GND")
+	)
+	(via
 		(at 203.25 151.8)
 		(size 0.5)
@@
 		(capping no)
 		(covering
+			(front no)
+			(back no)
+		)
+		(plugging
+			(front no)
+			(back no)
+		)
+		(filling no)
+		(net "GND")
+	)
+	(via
+		(at 165 130.5)
+		(size 0.5)
+		(drill 0.3)
+		(layers "F.Cu" "B.Cu")
+		(free yes)
+		(capping no)
+		(covering

Commit message: Update part values and BOM metadata
Parts:
- R1, R8: value 10k -> 5k
- R10, R3: value 5k -> 10k
- R13, R6: value 360 -> 1.8k
- R2, R4: value 3k -> 1.5k
- U24, U29: value AD8421 -> INA826AID
Changed lines of the file:
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@@
 			)
 		)
-		(property "Value" "10k"
+		(property "Value" "5k"
 			(at 0 1.43 0)
 			(layer "F.Fab")
@@
 			)
 		)
-		(property "Description" "RESISTOR:   SMD 0603 10kΩ ±0.1% 0.100W   [RG1608P-103-B-T5] [SMD]"
+		(property "Description" "RESISTOR:   SMD 0603 4.99kΩ ±0.1% 0.100W   [RG1608P-4991-B-T5] [SMD]"
 			(at 0 0 0)
 			(unlocked yes)
@@
 			)
 		)
-		(property "MPN" "RG1608P-103-B-T5"
+		(property "MPN" "RG1608P-4991-B-T5"
 			(at 0 0 0)
 			(unlocked yes)
@@
 			)
 		)
-		(property "OEPSPN" "OEPS020235"
+		(property "OEPSPN" "OEPS020233"
 			(at 0 0 0)
 			(unlocked yes)
@@
 			)
 		)
-		(property "Value" "3k"
+		(property "Value" "1.5k"
 			(at 0 1.43 90)
 			(layer "F.Fab")
@@
 			)
 		)
-		(property "Description" "RESISTOR:   SMD 0603 3kΩ ±0.1% 0.100W   [RG1608P-302-B-T5] [SMD]"
+		(property "Description" "RESISTOR:   SMD 0603 1.5kΩ ±0.1% 0.100W   [RG1608P-152-B-T5] [SMD]"
 			(at 0 0 270)
 			(unlocked yes)
@@
 			)
 		)
-		(property "Tolerance" "1%"
+		(property "Tolerance" "0.1%"
 			(at 0 0 270)
 			(unlocked yes)
@@
 			)
 		)
-		(property "MPN" "RG1608P-302-B-T5"
+		(property "MPN" "RG1608P-152-B-T5"
 			(at 0 0 270)
 			(unlocked yes)
@@
 			)
 		)
-		(property "OEPSPN" "OEPS020234"
+		(property "OEPSPN" "OEPS020262"
 			(at 0 0 270)
 			(unlocked yes)
@@
 			)
 		)
-		(property "Value" "360"
+		(property "Value" "1.8k"
 			(at 5.4716 -0.0476 90)
 			(layer "F.Fab")
@@
 			)
 		)
-		(property "Description" "RESISTOR:   SMD 0603 360Ω ±0.1% 0.100W   [RG1608P-361-B-T5] [SMD]"
+		(property "Description" "RESISTOR:   SMD 0603 1.8kΩ ±0.1% 0.100W   [RG1608P-182-B-T5] [SMD]"
 			(at 0 0 90)
 			(unlocked yes)
@@
 			)
 		)
-		(property "MPN" "RG1608P-361-B-T5"
+		(property "MPN" "RG1608P-182-B-T5 "
 			(at 0 0 90)
 			(unlocked yes)
@@
 			)
 		)
-		(property "OEPSPN" "OEPS020231"
+		(property "OEPSPN" "OEPS020261"
 			(at 0 0 90)
 			(unlocked yes)
@@
 			)
 		)
-		(property "Value" "5k"
+		(property "Value" "10k"
 			(at 0 1.43 90)
 			(layer "F.Fab")
@@
 			)
 		)
-		(property "Description" "RESISTOR:   SMD 0603 4.99kΩ ±0.1% 0.100W   [RG1608P-4991-B-T5] [SMD]"
+		(property "Description" "RESISTOR:   SMD 0603 10kΩ ±0.1% 0.100W   [RG1608P-103-B-T5] [SMD]"
 			(at 0 0 90)
 			(unlocked yes)
@@
 			)
 		)
-		(property "MPN" "RG1608P-4991-B-T5"
+		(property "MPN" "RG1608P-103-B-T5"
 			(at 0 0 90)
 			(unlocked yes)
@@
 			)
 		)
-		(property "OEPSPN" "OEPS020233"
+		(property "OEPSPN" "OEPS020235"
 			(at 0 0 90)
 			(unlocked yes)
@@
 			)
 		)
-		(property "Value" "3k"
+		(property "Value" "1.5k"
 			(at 0 1.43 90)
 			(layer "F.Fab")
@@
 			)
 		)
-		(property "Description" "RESISTOR:   SMD 0603 3kΩ ±0.1% 0.100W   [RG1608P-302-B-T5] [SMD]"
+		(property "Description" "RESISTOR:   SMD 0603 1.5kΩ ±0.1% 0.100W   [RG1608P-152-B-T5] [SMD]"
 			(at 0 0 270)
 			(unlocked yes)
@@
 			)
 		)
-		(property "Tolerance" "1%"
+		(property "Tolerance" "0.1%"
 			(at 0 0 270)
 			(unlocked yes)
@@
 			)
 		)
-		(property "MPN" "RG1608P-302-B-T5"
+		(property "MPN" "RG1608P-152-B-T5"
 			(at 0 0 270)
 			(unlocked yes)
@@
 			)
 		)
-		(property "OEPSPN" "OEPS020234"
+		(property "OEPSPN" "OEPS020262"
 			(at 0 0 270)
 			(unlocked yes)
@@
 			)
 		)
-		(property "Value" "5k"
+		(property "Value" "10k"
 			(at 0 1.43 90)
 			(layer "F.Fab")
@@
 			)
 		)
-		(property "Description" "RESISTOR:   SMD 0603 4.99kΩ ±0.1% 0.100W   [RG1608P-4991-B-T5] [SMD]"
+		(property "Description" "RESISTOR:   SMD 0603 10kΩ ±0.1% 0.100W   [RG1608P-103-B-T5] [SMD]"
 			(at 0 0 90)
 			(unlocked yes)
@@
 			)
 		)
-		(property "MPN" "RG1608P-4991-B-T5"
+		(property "MPN" "RG1608P-103-B-T5"
 			(at 0 0 90)
 			(unlocked yes)
@@
 			)
 		)
-		(property "OEPSPN" "OEPS020233"
+		(property "OEPSPN" "OEPS020235"
 			(at 0 0 90)
 			(unlocked yes)
@@
 			)
 		)
-		(property "Value" "360"
+		(property "Value" "1.8k"
 			(at 5.4716 -0.0476 90)
 			(layer "F.Fab")
@@
 			)
 		)
-		(property "Description" "RESISTOR:   SMD 0603 360Ω ±0.1% 0.100W   [RG1608P-361-B-T5] [SMD]"
+		(property "Description" "RESISTOR:   SMD 0603 1.8kΩ ±0.1% 0.100W   [RG1608P-182-B-T5] [SMD]"
 			(at 0 0 90)
 			(unlocked yes)
@@
 			)
 		)
-		(property "MPN" "RG1608P-361-B-T5"
+		(property "MPN" "RG1608P-182-B-T5 "
 			(at 0 0 90)
 			(unlocked yes)
@@
 			)
 		)
-		(property "OEPSPN" "OEPS020231"
+		(property "OEPSPN" "OEPS020261"
 			(at 0 0 90)
 			(unlocked yes)
@@
 			)
 		)
-		(property "Value" "10k"
+		(property "Value" "5k"
 			(at 0 1.43 0)
 			(layer "F.Fab")
@@
 			)
 		)
-		(property "Description" "RESISTOR:   SMD 0603 10kΩ ±0.1% 0.100W   [RG1608P-103-B-T5] [SMD]"
+		(property "Description" "RESISTOR:   SMD 0603 4.99kΩ ±0.1% 0.100W   [RG1608P-4991-B-T5] [SMD]"
 			(at 0 0 0)
 			(unlocked yes)
@@
 			)
 		)
-		(property "MPN" "RG1608P-103-B-T5"
+		(property "MPN" "RG1608P-4991-B-T5"
 			(at 0 0 0)
 			(unlocked yes)
@@
 			)
 		)
-		(property "OEPSPN" "OEPS020235"
+		(property "OEPSPN" "OEPS020233"
 			(at 0 0 0)
 			(unlocked yes)
@@
 			)
 		)
-		(property "Value" "AD8421"
+		(property "Value" "INA826AID"
 			(at 0 3.4 0)
 			(layer "F.Fab")
@@
 			)
 		)
-		(property "Description" "IC:   INST AMP 1 CIRCUIT   [AD8421BRZ-R7] [8-SOIC]"
+		(property "Description" "IC:   INST AMP 1 CIRCUIT   [INA826AIDR] [8-SOIC]"
 			(at 0 0 0)
 			(layer "F.Fab")
@@
 			)
 		)
-		(property "MPN" "AD8421BRZ-R7"
+		(property "MPN" "INA826AIDR"
 			(at 0 0 0)
 			(unlocked yes)
@@
 			)
 		)
-		(property "OEPSPN" "OEPS080222"
+		(property "OEPSPN" "OEPS080248"
 			(at 0 0 0)
 			(unlocked yes)
@@
 			)
 		)
-		(property "Value" "AD8421"
+		(property "Value" "INA826AID"
 			(at 0 3.4 0)
 			(layer "F.Fab")
@@
 			)
 		)
-		(property "Description" "IC:   INST AMP 1 CIRCUIT   [AD8421BRZ-R7] [8-SOIC]"
+		(property "Description" "IC:   INST AMP 1 CIRCUIT   [INA826AIDR] [8-SOIC]"
 			(at 0 0 0)
 			(layer "F.Fab")
@@
 			)
 		)
-		(property "MPN" "AD8421BRZ-R7"
+		(property "MPN" "INA826AIDR"
 			(at 0 0 0)
 			(unlocked yes)
@@
 			)
 		)
-		(property "OEPSPN" "OEPS080222"
+		(property "OEPSPN" "OEPS080248"
 			(at 0 0 0)
 			(unlocked yes)
@@
 			)
 		)
-		(property "Description" "CONNECTOR:   USB2.0 TYPE C 24P SMD R/A   [USB4105-GF-A] [SMD/TH]"
+		(property "Description" "CONNECTOR:   USB2.0 TYPE C 16P SMD R/A   [USB4105-GF-A] [SMD/TH]"
 			(at 0 0 0)
 			(unlocked yes)
