File: PCB/mcu.kicad_sch (KiCad schematic)
At the start: 59 parts, among them J1 302-R161, J2 0731375003, J3 0731375003, SW2 PTS645VH58-2 LFS, SW3 TS04-66-50-BK-160-SMT, U25 W25Q128JVS, U30 RP2354B, Y1 ABM8AIG-12.000MHZ-12-2Z-T3

Commit message: Add OEPS PN to main PCB
Parts:
- C55, C56, C57, C58, C59, C60, C61, C64, C81, C83, C84: MPN (none) -> C1005X7R1E104K050BB; OEPSPN (none) -> OEPS010050
- C62: MPN (none) -> C1005X7R1E104K050BB; OEPSPN (none) -> OEPS010050; TempCo (none) -> X7R
- C70, C71: MPN (none) -> CL05C220JB51PNC; OEPSPN (none) -> OEPS010080
- C85, C87, C88: MPN (none) -> KGM05CR51C475MH; OEPSPN (none) -> OEPS010097
- C86: MPN (none) -> KGM05CR51C475MH; OEPSPN (none) -> OEPS010097; TempCo (none) -> X5R
- D1, D10, D11, D12, D13, D14, D15, D16, D6, D8: MPN (none) -> BAT54SW; OEPSPN (none) -> OEPS030056
- D4, D5: OEPSPN (none) -> OEPS030055
- J1: OEPSPN (none) -> OEPS070152
- J2, J3: OEPSPN (none) -> OEPS070151
- L1: OEPSPN (none) -> OEPS040036
- R15, R32: MPN (none) -> RC0603FR-0710KL; OEPSPN (none) -> OEPS020133
- R16, R21, R22, R23, R24, R25, R36, R37, R38, R39: MPN TNPW1206100RBEEA -> CRCW0805270RFKEAHP; OEPSPN OEPS020172 -> OEPS020024
- R27: MPN (none) -> RG1608P-102-B-T5; OEPSPN (none) -> OEPS020215
- R28, R29: MPN (none) -> CRCW0603100RFKEAHP; OEPSPN (none) -> OEPS020042
- R30, R31, R33: MPN (none) -> RMCF0402FT27R0; OEPSPN (none) -> OEPS020170
- R34, R35: MPN (none) -> RC0603FR-07200RL; OEPSPN (none) -> OEPS020141
- SW2: OEPSPN (none) -> OEPS070114
- SW3: OEPSPN (none) -> OEPS070115
- U25: MPN W25Q128JVS -> W25Q128JVSIQ; OEPSPN (none) -> OEPS080163
- U30: MPN (none) -> SC1512-A4; OEPSPN (none) -> OEPS080220
- Y1: OEPSPN (none) -> OEPS100059
