File: PCB/stimjim.kicad_sch (KiCad schematic)
At the start: 22 parts, among them J10 USB4105-GF-A, J11 BM03B-SRSS-TB, J4 10129383-910002ALF, U151 AP2112K-3.3

Commit message: Exclude test points from assembly position files
Exclude test points (TPs), mounting holes (H1-H4), and mounting pads (MP1-MP2) from position files used for PCB assembly. These are non-assembly components that should not be included in pick-and-place machine files.

If possible, the Attributes for Test Points and Mounting Holes should be:
[X]  Exclude from bill of materials
[  ]  Exclude from board
[X]  Exclude from position files
[  ]  Do not populate
Parts:
- MP1, N2: now left out of the parts list
Changed lines of the file:
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@@
 		(in_bom no)
 		(on_board yes)
-		(in_pos_files yes)
+		(in_pos_files no)
 		(dnp no)
 		(property "Reference" "H1"
@@
 		(in_bom no)
 		(on_board yes)
-		(in_pos_files yes)
+		(in_pos_files no)
 		(dnp no)
 		(property "Reference" "H2"
@@
 		(in_bom no)
 		(on_board yes)
-		(in_pos_files yes)
+		(in_pos_files no)
 		(dnp no)
 		(property "Reference" "H3"
@@
 		(in_bom no)
 		(on_board yes)
-		(in_pos_files yes)
+		(in_pos_files no)
 		(dnp no)
 		(property "Reference" "H4"
@@
 		(in_bom no)
 		(on_board yes)
-		(in_pos_files yes)
+		(in_pos_files no)
 		(dnp no)
 		(property "Reference" "TP56"
@@
 		(in_bom no)
 		(on_board yes)
-		(in_pos_files yes)
+		(in_pos_files no)
 		(dnp no)
 		(fields_autoplaced yes)
@@
 		(in_bom no)
 		(on_board yes)
-		(in_pos_files yes)
+		(in_pos_files no)
 		(dnp no)
 		(property "Reference" "TP53"
@@
 		(in_bom no)
 		(on_board yes)
-		(in_pos_files yes)
+		(in_pos_files no)
 		(dnp no)
 		(property "Reference" "TP54"
@@
 		(body_style 1)
 		(exclude_from_sim no)
-		(in_bom yes)
+		(in_bom no)
 		(on_board no)
-		(in_pos_files yes)
+		(in_pos_files no)
 		(dnp no)
 		(property "Reference" "MP1"
@@
 		(body_style 1)
 		(exclude_from_sim no)
-		(in_bom yes)
+		(in_bom no)
 		(on_board no)
-		(in_pos_files yes)
+		(in_pos_files no)
 		(dnp no)
 		(fields_autoplaced yes)

Commit message: Add OEPS PN to main PCB
Parts:
- C295, C297: MPN (none) -> CL10A105KA8NNNC; OEPSPN (none) -> OEPS010022
- D3: OEPSPN (none) -> OEPS030055
- D9: MPN TPD4E05U06DQA -> TPD4E05U06DQAR; OEPSPN (none) -> OEPS030037
- J10: OEPSPN (none) -> OEPS070105
- J11: OEPSPN (none) -> OEPS070121
- J4: OEPSPN (none) -> OEPS070120
- N1: value SMTRA_M3-7-5ET -> SMTRAM3-7-5ET; MPN SMTRA_M3-7-5ET -> SMTRAM3-7-5ET; OEPSPN (none) -> OEPS100089
- R26: MPN (none) -> RC0603FR-07200RL; OEPSPN (none) -> OEPS020141
- R266, R267: MPN (none) -> ERJ-2RKF5101X; OEPSPN (none) -> OEPS020173
- U151: MPN AP2112K-3.3 -> AP2112K-3.3TRG1; OEPSPN (none) -> OEPS080155
Changed lines of the file:
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@@
 			)
 		)
-		(property "Description" "Light emitting diode"
+		(property "Description" "DIODE:   LED TH Green 565nm 20mA R/A   [SSF-LXH100GD-01] [TH]"
 			(at 154.94 135.89 0)
 			(hide yes)
@@
 			)
 		)
+		(property "OEPSPN" "OEPS030055"
+			(at 154.94 135.89 0)
+			(hide yes)
+			(show_name no)
+			(do_not_autoplace no)
+			(effects
+				(font
+					(size 1.27 1.27)
+				)
+			)
+		)
 		(pin "1"
 		)
@@
 			)
 		)
-		(property "Value" "SMTRA_M3-7-5ET"
+		(property "Value" "SMTRAM3-7-5ET"
 			(at 191.77 152.3999 0)
 			(show_name no)
@@
 			)
 		)
-		(property "Description" "Mounting Hole with connection"
+		(property "Description" "OTHER:   SURFACE MOUNT R'ANGLE M3   [SMTRAM3-7-5ET] [Other]"
 			(at 189.23 152.4 0)
 			(hide yes)
@@
 			)
 		)
-		(property "MPN" "SMTRA_M3-7-5ET"
+		(property "MPN" "SMTRAM3-7-5ET"
+			(at 189.23 152.4 0)
+			(hide yes)
+			(show_name no)
+			(do_not_autoplace no)
+			(effects
+				(font
+					(size 1.27 1.27)
+				)
+			)
+		)
+		(property "OEPSPN" "OEPS100089"
 			(at 189.23 152.4 0)
 			(hide yes)
@@
 			)
 		)
-		(property "Description" "USB 2.0-only 16P Type-C Receptacle connector"
+		(property "Description" "CONNECTOR:   USB2.0 TYPE C 24P SMD R/A   [USB4105-GF-A] [SMD/TH]"
 			(at 46.99 60.96 0)
 			(hide yes)
@@
 			)
 		)
+		(property "OEPSPN" "OEPS070105"
+			(at 46.99 60.96 0)
+			(hide yes)
+			(show_name no)
+			(do_not_autoplace no)
+			(effects
+				(font
+					(size 1.27 1.27)
+				)
+			)
+		)
 		(pin "A1"
 		)
@@
 			)
 		)
-		(property "Description" "Unpolarized capacitor"
+		(property "Description" "CAPACITOR:   SMD CER 0603 1uF 25V ±10% X5R   [CL10A105KA8NNNC] [SMD]"
 			(at 138.43 127 0)
 			(hide yes)
@@
 			)
 		)
-		(property "MPN" ""
+		(property "MPN" "CL10A105KA8NNNC"
+			(at 138.43 127 0)
+			(hide yes)
+			(show_name no)
+			(do_not_autoplace no)
+			(effects
+				(font
+					(size 1.27 1.27)
+				)
+			)
+		)
+		(property "OEPSPN" "OEPS010022"
 			(at 138.43 127 0)
 			(hide yes)
@@
 			)
 		)
-		(property "Description" "Generic connector, single row, 01x03, script generated (kicad-library-utils/schlib/autogen/connector/)"
+		(property "Description" "CONNECTOR:   HEADER VERT 3POS 1MM   [BM03B-SRSS-TB] [SMD]"
 			(at 242.57 119.38 0)
 			(hide yes)
@@
 			)
 		)
+		(property "OEPSPN" "OEPS070121"
+			(at 242.57 119.38 0)
+			(hide yes)
+			(show_name no)
+			(do_not_autoplace no)
+			(effects
+				(font
+					(size 1.27 1.27)
+				)
+			)
+		)
 		(pin "2"
 		)
@@
 			)
 		)
-		(property "Description" "Unpolarized capacitor"
+		(property "Description" "CAPACITOR:   SMD CER 0603 1uF 25V ±10% X5R   [CL10A105KA8NNNC] [SMD]"
 			(at 101.6 125.73 0)
 			(hide yes)
@@
 			)
 		)
-		(property "MPN" ""
+		(property "MPN" "CL10A105KA8NNNC"
+			(at 101.6 125.73 0)
+			(hide yes)
+			(show_name no)
+			(do_not_autoplace no)
+			(effects
+				(font
+					(size 1.27 1.27)
+				)
+			)
+		)
+		(property "OEPSPN" "OEPS010022"
 			(at 101.6 125.73 0)
 			(hide yes)
@@
 			)
 		)
-		(property "Description" "4-Channel ESD Protection for Super-Speed USB 3.0 Interface, USON-10"
+		(property "Description" "DIODE:   TVS DIODE 5.5VWM 14VC   [TPD4E05U06DQAR] [10-UFDFN]"
 			(at 124.46 76.2 0)
 			(hide yes)
@@
 			)
 		)
-		(property "MPN" "TPD4E05U06DQA"
+		(property "MPN" "TPD4E05U06DQAR"
+			(at 124.46 76.2 0)
+			(hide yes)
+			(show_name no)
+			(do_not_autoplace no)
+			(effects
+				(font
+					(size 1.27 1.27)
+				)
+			)
+		)
+		(property "OEPSPN" "OEPS030037"
 			(at 124.46 76.2 0)
 			(hide yes)
@@
 			)
 		)
-		(property "Description" "Resistor, US symbol"
+		(property "Description" "RESISTOR:   SMD 0402 5.1kΩ ±1% 0.100W   [ERJ-2RKF5101X] [SMD]"
 			(at 88.9 76.2 0)
 			(hide yes)
@@
 			)
 		)
-		(property "MPN" ""
+		(property "MPN" "ERJ-2RKF5101X"
+			(at 88.9 76.2 90)
+			(hide yes)
+			(show_name no)
+			(do_not_autoplace no)
+			(effects
+				(font
+					(size 1.27 1.27)
+				)
+			)
+		)
+		(property "OEPSPN" "OEPS020173"
 			(at 88.9 76.2 90)
 			(hide yes)
@@
 			)
 		)
-		(property "Description" "600mA low dropout linear regulator, with enable pin, 3.8V-6V input voltage range, 3.3V fixed positive output, SOT-23-5"
+		(property "Description" "IC:   LDO 3.3V 600mA   [AP2112K-3.3TRG1] [SOT-23-5]"
 			(at 121.92 123.19 0)
 			(hide yes)
@@
 			)
 		)
-		(property "MPN" "AP2112K-3.3"
+		(property "MPN" "AP2112K-3.3TRG1"
+			(at 121.92 123.19 0)
+			(hide yes)
+			(show_name no)
+			(do_not_autoplace no)
+			(effects
+				(font
+					(size 1.27 1.27)
+				)
+			)
+		)
+		(property "OEPSPN" "OEPS080155"
 			(at 121.92 123.19 0)
 			(hide yes)
@@
 			)
 		)
-		(property "Description" "Generic connector, double row, 02x04, odd/even pin numbering scheme (row 1 odd numbers, row 2 even numbers), script generated (kicad-library-utils/schlib/autogen/connector/)"
+		(property "Description" "CONNECTOR:   HEADER VERT 2x5POS 2.54MM   [10129383-910002ALF] [SMD]"
 			(at 252.73 104.14 0)
 			(hide yes)
@@
 			)
 		)
+		(property "OEPSPN" "OEPS070120"
+			(at 252.73 104.14 0)
+			(hide yes)
+			(show_name no)
+			(do_not_autoplace no)
+			(effects
+				(font
+					(size 1.27 1.27)
+				)
+			)
+		)
 		(pin "1"
 		)
@@
 			)
 		)
-		(property "Description" "Resistor, US symbol"
+		(property "Description" "RESISTOR:   SMD 0603 200Ω ±1% 0.100W (OEPS J30 017)   [RC0603FR-07200RL] [SMD]"
 			(at 154.94 127 0)
 			(hide yes)
@@
 			)
 		)
-		(property "MPN" ""
+		(property "MPN" "RC0603FR-07200RL"
+			(at 154.94 127 90)
+			(hide yes)
+			(show_name no)
+			(do_not_autoplace no)
+			(effects
+				(font
+					(size 1.27 1.27)
+				)
+			)
+		)
+		(property "OEPSPN" "OEPS020141"
 			(at 154.94 127 90)
 			(hide yes)
@@
 			)
 		)
-		(property "Description" "Resistor, US symbol"
+		(property "Description" "RESISTOR:   SMD 0402 5.1kΩ ±1% 0.100W   [ERJ-2RKF5101X] [SMD]"
 			(at 80.01 76.2 0)
 			(hide yes)
@@
 			)
 		)
-		(property "MPN" ""
+		(property "MPN" "ERJ-2RKF5101X"
+			(at 80.01 76.2 90)
+			(hide yes)
+			(show_name no)
+			(do_not_autoplace no)
+			(effects
+				(font
+					(size 1.27 1.27)
+				)
+			)
+		)
+		(property "OEPSPN" "OEPS020173"
 			(at 80.01 76.2 90)
 			(hide yes)
