File: PCB/channel.kicad_sch (KiCad schematic)
At the start: 78 parts, among them J9 0731375003, U1 OPA197, U10 OPA197, U13 CC3-0512DF-E, U14 ISO7760, U15 ISO7741, U16 MC78L05ACDR2G, U17 AD5752, U18 AD7321, U19 AD1582, U20 OPA197, U23 DG409DYZ-T, U24 AD8421, U27 LT1995

Commit message: Add OEPS PN to main PCB
Parts:
- C19, C21: MPN (none) -> C1608X7R1H103K080AA; OEPSPN (none) -> OEPS010074
- C26, C27, C31, C32, C34, C35, C38, C39, C41, C42, C43, C44, C47, C48, C49, C50, C63, C66, C80, C89: MPN (none) -> GRM188R72A104KA35D; OEPSPN (none) -> OEPS010009
- C28, C29, C30: MPN (none) -> GRT319R6YA106KE01D; OEPSPN (none) -> OEPS010094
- C33, C36, C37, C40, C52: MPN (none) -> CL10A105KA8NNNC; OEPSPN (none) -> OEPS010022; TempCo (none) -> X5R
- C54: MPN (none) -> DNP; OEPSPN (none) -> OEPS000000
- C68, C72, C74, C76: MPN (none) -> GRM188R6YA106MA73J; OEPSPN (none) -> OEPS010093
- C78: MPN (none) -> C0603C100J5GACTU; OEPSPN (none) -> OEPS010096
- C91, C93: MPN (none) -> GRM188R61E475KE11D; OEPSPN (none) -> OEPS010047
- J9: OEPSPN (none) -> OEPS070151
- R10: MPN (none) -> RG1608P-4991-B-T5; OEPSPN (none) -> OEPS020233
- R12: MPN (none) -> RG1608P-101-B-T5; OEPSPN (none) -> OEPS020232
- R13: MPN (none) -> RG1608P-361-B-T5; OEPSPN (none) -> OEPS020231
- R14: MPN (none) -> RG1608P-102-B-T5; OEPSPN (none) -> OEPS020215
- R18: MPN (none) -> RC0603FR-0710KL; OEPSPN (none) -> OEPS020133; Tolerance 1% -> (none)
- R2: MPN (none) -> RG1608P-302-B-T5; OEPSPN (none) -> OEPS020234
- R20: MPN (none) -> CRGCQ1210J2M2; OEPSPN (none) -> OEPS020230
- R8: MPN (none) -> RG1608P-103-B-T5; OEPSPN (none) -> OEPS020235
- R9: MPN (none) -> RCS06030000Z0EA; OEPSPN (none) -> OEPS020151
- U1, U10, U20: MPN OPA197IDR -> OPA197IDR; OEPSPN (none) -> OEPS080229
- U13: OEPSPN (none) -> OEPS100043
- U14: MPN ISO7760DWR -> ISO7760DWR; OEPSPN (none) -> OEPS080228
- U15: OEPSPN (none) -> OEPS080227
- U16: OEPSPN (none) -> OEPS080226
- U17: OEPSPN (none) -> OEPS080091
- U18: MPN AD7321BRUZ-REEL7 -> AD7321BRUZ-REEL7; OEPSPN (none) -> OEPS080225
- U19: MPN AD1582ARTZ-REEL -> AD1582ARTZ-REEL7; OEPSPN (none) -> OEPS080224
- U23: OEPSPN (none) -> OEPS080223
- U24: MPN (none) -> AD8421BRZ-R7; OEPSPN (none) -> OEPS080222
- U27: MPN (none) -> LT1995CMS#PBF; OEPSPN (none) -> OEPS080221

Commit message: Add ground connections to rp2354 thermal pad
- It was floating
- Fix some silkscreen issues
Changed lines of the file:
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@@
 	(text "DAC"
 		(exclude_from_sim no)
-		(at 106.68 75.946 0)
+		(at 110.998 75.946 0)
 		(effects
 			(font

Commit message: Update part values and BOM metadata
Parts:
- R10: value 5k -> 10k; MPN RG1608P-4991-B-T5 -> RG1608P-103-B-T5; OEPSPN OEPS020233 -> OEPS020235
- R13: value 360 -> 1.8k; MPN RG1608P-361-B-T5 -> RG1608P-182-B-T5; OEPSPN OEPS020231 -> OEPS020261
- R2: value 3k -> 1.5k; MPN RG1608P-302-B-T5 -> RG1608P-152-B-T5; OEPSPN OEPS020234 -> OEPS020262; Tolerance 1% -> 0.1%
- R8: value 10k -> 5k; MPN RG1608P-103-B-T5 -> RG1608P-4991-B-T5; OEPSPN OEPS020235 -> OEPS020233
- U24: value AD8421 -> INA826AID; MPN AD8421BRZ-R7 -> INA826AIDR; OEPSPN OEPS080222 -> OEPS080248
Changed lines of the file:
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@@
 			)
 		)
-		(property "Value" "3k"
+		(property "Value" "1.5k"
 			(at 213.36 72.39 90)
 			(show_name no)
@@
 			)
 		)
-		(property "Description" "RESISTOR:   SMD 0603 3kΩ ±0.1% 0.100W   [RG1608P-302-B-T5] [SMD]"
+		(property "Description" "RESISTOR:   SMD 0603 1.5kΩ ±0.1% 0.100W   [RG1608P-152-B-T5] [SMD]"
 			(at 213.36 76.2 0)
 			(hide yes)
@@
 			)
 		)
-		(property "Tolerance" "1%"
+		(property "Tolerance" "0.1%"
 			(at 213.36 76.2 90)
 			(hide yes)
@@
 			)
 		)
-		(property "MPN" "RG1608P-302-B-T5"
+		(property "MPN" "RG1608P-152-B-T5"
 			(at 213.36 76.2 90)
 			(hide yes)
@@
 			)
 		)
-		(property "OEPSPN" "OEPS020234"
+		(property "OEPSPN" "OEPS020262"
 			(at 213.36 76.2 90)
 			(hide yes)
@@
 			)
 		)
-		(property "Value" "10k"
+		(property "Value" "5k"
 			(at 229.87 39.0144 90)
 			(show_name no)
@@
 			)
 		)
-		(property "Description" "RESISTOR:   SMD 0603 10kΩ ±0.1% 0.100W   [RG1608P-103-B-T5] [SMD]"
+		(property "Description" "RESISTOR:   SMD 0603 4.99kΩ ±0.1% 0.100W   [RG1608P-4991-B-T5] [SMD]"
 			(at 229.87 41.91 0)
 			(hide yes)
@@
 			)
 		)
-		(property "MPN" "RG1608P-103-B-T5"
+		(property "MPN" "RG1608P-4991-B-T5"
 			(at 229.87 41.91 90)
 			(hide yes)
@@
 			)
 		)
-		(property "OEPSPN" "OEPS020235"
+		(property "OEPSPN" "OEPS020233"
 			(at 229.87 41.91 90)
 			(hide yes)
@@
 			)
 		)
-		(property "Value" "AD8421"
+		(property "Value" "INA826AID"
 			(at 270.51 67.2398 0)
 			(show_name no)
@@
 			)
 		)
-		(property "Description" "IC:   INST AMP 1 CIRCUIT   [AD8421BRZ-R7] [8-SOIC]"
+		(property "Description" "IC:   INST AMP 1 CIRCUIT   [INA826AIDR] [8-SOIC]"
 			(at 255.27 71.12 0)
 			(hide yes)
@@
 			)
 		)
-		(property "MPN" "AD8421BRZ-R7"
+		(property "MPN" "INA826AIDR"
 			(at 255.27 71.12 0)
 			(hide yes)
@@
 			)
 		)
-		(property "OEPSPN" "OEPS080222"
+		(property "OEPSPN" "OEPS080248"
 			(at 255.27 71.12 0)
 			(hide yes)
@@
 			)
 		)
-		(property "Value" "360"
+		(property "Value" "1.8k"
 			(at 238.3028 72.263 0)
 			(show_name no)
@@
 			)
 		)
-		(property "Description" "RESISTOR:   SMD 0603 360Ω ±0.1% 0.100W   [RG1608P-361-B-T5] [SMD]"
+		(property "Description" "RESISTOR:   SMD 0603 1.8kΩ ±0.1% 0.100W   [RG1608P-182-B-T5] [SMD]"
 			(at 240.03 71.12 0)
 			(hide yes)
@@
 			)
 		)
-		(property "MPN" "RG1608P-361-B-T5"
+		(property "MPN" "RG1608P-182-B-T5 "
 			(at 240.03 71.12 0)
 			(hide yes)
@@
 			)
 		)
-		(property "OEPSPN" "OEPS020231"
+		(property "OEPSPN" "OEPS020261"
 			(at 240.03 71.12 0)
 			(hide yes)
@@
 			)
 		)
-		(property "Value" "5k"
+		(property "Value" "10k"
 			(at 254 39.0144 90)
 			(show_name no)
@@
 			)
 		)
-		(property "Description" "RESISTOR:   SMD 0603 4.99kΩ ±0.1% 0.100W   [RG1608P-4991-B-T5] [SMD]"
+		(property "Description" "RESISTOR:   SMD 0603 10kΩ ±0.1% 0.100W   [RG1608P-103-B-T5] [SMD]"
 			(at 254 41.91 0)
 			(hide yes)
@@
 			)
 		)
-		(property "MPN" "RG1608P-4991-B-T5"
+		(property "MPN" "RG1608P-103-B-T5"
 			(at 254 41.91 90)
 			(hide yes)
@@
 			)
 		)
-		(property "OEPSPN" "OEPS020233"
+		(property "OEPSPN" "OEPS020235"
 			(at 254 41.91 90)
 			(hide yes)
