File: PCB/channel.kicad_sch (KiCad schematic)
At the start: 78 parts, among them J9 0731375003, U1 OPA197, U10 OPA197, U13 CC3-0512DF-E, U14 ISO7760, U15 ISO7741, U16 MC78L05ACDR2G, U17 AD5752, U18 AD7321, U19 AD1582, U20 OPA197, U23 DG409DYZ-T, U24 INA826AID, U27 LT1995

Commit message: Update 5k resistor part references
Switch the 5k 0603 precision resistor references from RG1608P-4991-B-T5 to RT0603BRE075KL in the schematic, PCB, and BOM.
Parts:
- R8: MPN RG1608P-4991-B-T5 -> RT0603BRE075KL; OEPSPN OEPS020233 -> OEPS020263
Changed lines of the file:
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@@
 			)
 		)
-		(property "Description" "RESISTOR:   SMD 0603 4.99kΩ ±0.1% 0.100W   [RG1608P-4991-B-T5] [SMD]"
+		(property "Description" "RESISTOR:   SMD 0603 5kΩ ±0.1% 0.100W   [RT0603BRE075KL] [SMD]"
 			(at 229.87 41.91 0)
 			(hide yes)
@@
 			)
 		)
-		(property "MPN" "RG1608P-4991-B-T5"
+		(property "MPN" "RT0603BRE075KL"
 			(at 229.87 41.91 90)
 			(hide yes)
@@
 			)
 		)
-		(property "OEPSPN" "OEPS020233"
+		(property "OEPSPN" "OEPS020263"
 			(at 229.87 41.91 90)
 			(hide yes)

Commit message: Update AD1582 voltage reference part
This changes the AD1582 voltage reference from the ARTZ variant to the BRTZ precision variant.
Parts:
- U19: MPN AD1582ARTZ-REEL7 -> AD1582BRTZ-REEL7; OEPSPN OEPS080224 -> OEPS080250
Changed lines of the file:
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@@
 			)
 		)
-		(property "Description" "IC:   VREF 2.5V 0.8% 5mA   [AD1582ARTZ-REEL7] [SOT-23-3]"
+		(property "Description" "IC:   VREF 2.5V 0.08% 5mA   [AD1582BRTZ-REEL7] [SOT-23-3]"
 			(at 139.7 40.64 0)
 			(hide yes)
@@
 			)
 		)
-		(property "MPN" "AD1582ARTZ-REEL7"
+		(property "MPN" "AD1582BRTZ-REEL7"
 			(at 139.7 40.64 0)
 			(hide yes)
@@
 			)
 		)
-		(property "OEPSPN" "OEPS080224"
+		(property "OEPSPN" "OEPS080250"
 			(at 139.7 40.64 0)
 			(hide yes)
