File: PCB/panels/panel-back.kicad_pcb (KiCad board)
At the start: 2 copper layers, 140 x 35 mm, 6 parts

Commit message: Add/edit silk screen and solder mask labels
Front panel:
- Add stimjim logo to solder mask
- Add "Dual isolated stimulus generator" to silk screen
Back panel:
- Shrink stimjim logo and center over usb cutout
- Add open ephys logo to solder mask
Parts:
- removed the G*** at (102.8, 51.4)
- added G***: LOGO, LOGO, F.Cu at (201.5, 72.5)
- added G***: LOGO, LOGO, F.Cu at (99.1, 55.0)
- added kibuzzard-69DFD1D5: G***, kibuzzard-69DFD1D5, F.Cu at (144.5, 50.5)
Other:
- board text removed: "AUX IO"
